Commit message: Fix Urdf 2

File: Hardware/CAD/Robot/urdf/robot_humanoid/urdf/robot_humanoid.urdf (robot description, URDF)
Before this commit: robot robot_humanoid, 19 links, 18 joints
Links:
- link ankle_ankle_right_link: mass 0.0859210745253493 -> 0.0859210745253492
- link base_hip_left_link: mass 0.107894198693898 -> 0.0540513645564241
- link base_hip_right_link: mass 0.107894198771709 -> 0.0540513645953296
- link base_link: mass 0.0025162912702426 -> 0.0483184538892821
- link hip_head_link: mass 1.9465439707667 -> 0.0591715303385524
- link hip_hip_left_link: mass 0.12988008385202 -> 0.0760372497010778
- link hip_hip_right_link: mass 0.129880083890925 -> 0.0760372497399833
- link hip_knee_left_link: mass 0.130204487068308 -> 0.0763616529153324
- link hip_knee_right_link: mass 0.130204487068308 -> 0.0763616529153324
- link hip_shoulder_left_link: mass 0.107894198733174 -> 0.054051364576062
- link hip_shoulder_right_link: mass 0.107894198733174 -> 0.054051364576062
- link knee_ankle_left_link: mass 0.0814463522717177 -> 0.0276035181342435
- link knee_ankle_right_link: mass 0.0276035181342435 -> 0.0226549246672409
- link knee_knee_left_link: mass 0.0850053645564242 -> 0.0850053645564241
- link shoulder_shoulder_left_link: mass 0.0772422226634494 -> 0.0772422226634493
- link shoulder_shoulder_right_link: mass 0.0772422226634494 -> 0.0772422226634495
Joints:
- joint base_hip_left_joint: axis 0 0 -1 -> 0 0 1; origin xyz=-0.0357002452027679 -0.0192546745613186 -0.0270000000000002 rpy=1.5707963267949 0 -0.0352246775973257 -> xyz=-0.0357002452027679 -0.0192546745613186 -0.0270000000000002 rpy=1.57079632679489 0 3.10636797599247
- joint base_hip_middle_joint: origin xyz=0 0 0.0048 rpy=0 0 0 -> xyz=0 0 0.00479999999999899 rpy=0 0 0
- joint hip_hip_left_joint: origin xyz=-0.0295000000000003 -0.0205000000000002 -0.0105000000000001 rpy=3.14159265358979 -1.5707963267949 0 -> xyz=0.0295000000000003 -0.0205000000000002 0.0105000000000001 rpy=0 1.5707963267949 0
- joint hip_shoulder_left_joint: axis 0 0 -1 -> 0 0 1; origin xyz=-0.108 0.0195000000000005 0.1093 rpy=1.5707963267949 0 3.14159265358979 -> xyz=-0.108 0.0195000000000005 0.1093 rpy=1.5707963267949 0 0
- joint shoulder_shoulder_left_joint: origin xyz=-0.0105000000000001 -0.0205 -0.0309 rpy=3.14159265358979 -1.5707963267949 0 -> xyz=0.0105000000000001 -0.0205 0.0309 rpy=0 1.5707963267949 0

Commit message: fix cad

File: Hardware/CAD/Robot/urdf/robot_humanoid/urdf/robot_humanoid.urdf (robot description, URDF)
Before this commit: robot robot_humanoid, 19 links, 18 joints
Links:
- link ankle_ankle_right_link: mass 0.0859210745253493 -> 0.085921
- link base_hip_left_link: mass 0.0540513645564241 -> 0.054051
- link base_hip_middle_link: mass 0.322024415361419 -> 0
- link base_hip_right_link: mass 0.0540513645953296 -> 0.054051
- link base_link: mass 0.0505669346650319 -> 0.050567
- link hip_head_link: mass 0.0602957707264273 -> 0.11435
- link hip_hip_left_link: mass 0.0782857304768276 -> 0.078286
- link hip_hip_right_link: mass 0.0782857305157331 -> 0.078286
- link hip_knee_left_link: mass 0.0763616529153324 -> 0.076362
- link hip_knee_right_link: mass 0.0763616529153324 -> 0.076362
- link hip_shoulder_left_link: mass 0.054051364576062 -> 0.054051
- link hip_shoulder_right_link: mass 0.054051364576062 -> 0.054051
- link knee_ankle_left_link: mass 0.0298519989099933 -> 0.029852
- link knee_ankle_right_link: mass 0.0249034054429908 -> 0.024903
- link knee_knee_left_link: mass 0.0850053645564241 -> 0.085005
- link shoulder_elbow_left_link: mass 0.054051364576062 -> 0.094735
- link shoulder_elbow_right_link: mass 0.054051364576062 -> 0.094683
- link shoulder_shoulder_left_link: mass 0.0794907034391991 -> 0.079491
- link shoulder_shoulder_right_link: mass 0.0794907034391993 -> 0.079491
Joints:
- joint ankle_ankle_right_joint: limit lower=0 upper=0 effort=0 velocity=0 -> lower=-1.2217 upper=1.2217 effort=1.08 velocity=6.16; origin xyz=0.0214999999999996 -0.0570000000000001 -0.0215000000000021 rpy=0 1.5707963267949 0 -> xyz=0.0215 -0.057 -0.0215 rpy=0 1.5708 0
- joint base_hip_left_joint: limit lower=0 upper=0 effort=0 velocity=0 -> lower=-0.69813 upper=0.17453 effort=1.08 velocity=6.16; origin xyz=-0.0357002452027679 -0.0192546745613186 -0.0270000000000002 rpy=1.57079632679489 0 3.10636797599247 -> xyz=-0.035 -0.0205 -0.027 rpy=1.5708 0 -3.1416
- joint base_hip_middle_joint: limit lower=0 upper=0 effort=0 velocity=0 -> lower=-0.5236 upper=0.5236 effort=1.08 velocity=6.16; origin xyz=0 0 0.00479999999999899 rpy=0 0 0 -> xyz=0 0 0.0048 rpy=0 0 0
- joint base_hip_right_joint: limit lower=0 upper=0 effort=0 velocity=0 -> lower=-0.69813 upper=0.17453 effort=1.08 velocity=6.16; origin xyz=0.0342563320604241 -0.0217198921214098 -0.0270000000000003 rpy=1.5707963267949 0 -0.0352246775973258 -> xyz=0.035 -0.0205 -0.027 rpy=1.5708 0 0
- joint hip_head_joint: origin xyz=0.00102807858096265 -0.00174999999999934 0.144615997868974 rpy=0 0 0 -> xyz=0.0010281 -0.00175 0.14462 rpy=0 0 0
- joint hip_hip_left_joint: limit lower=0 upper=0 effort=0 velocity=0 -> lower=-0.5236 upper=0.69813 effort=1.08 velocity=6.16; origin xyz=0.0295000000000003 -0.0205000000000002 0.0105000000000001 rpy=0 1.5707963267949 0 -> xyz=0.0295 -0.0205 0.0105 rpy=0 1.5708 0
- joint hip_hip_right_joint: limit lower=0 upper=0 effort=0 velocity=0 -> lower=-0.69813 upper=0.5236 effort=1.08 velocity=6.16; origin xyz=0.0308999999999979 -0.0204999999999999 -0.0125999999999999 rpy=0 1.5707963267949 0 -> xyz=0.0309 -0.0205 -0.0126 rpy=0 1.5708 0
- joint hip_knee_left_joint: limit lower=0 upper=0 effort=0 velocity=0 -> lower=-1.3963 upper=1.3963 effort=1.08 velocity=6.16; origin xyz=0 -0.0599999999999997 0 rpy=0 0 0 -> xyz=0 -0.06 0 rpy=0 0 0
- joint hip_knee_right_joint: limit lower=0 upper=0 effort=0 velocity=0 -> lower=-1.3963 upper=1.3963 effort=1.08 velocity=6.16; origin xyz=0 -0.0599999999999997 0 rpy=0 0 0 -> xyz=0 -0.06 0 rpy=0 0 0
- joint hip_shoulder_left_joint: limit lower=0 upper=0 effort=0 velocity=0 -> lower=-1.2217 upper=0.17453 effort=1.08 velocity=6.16; origin xyz=-0.108 0.0195000000000005 0.1093 rpy=1.5707963267949 0 0 -> xyz=-0.108 0.0195 0.1093 rpy=1.5708 0 0
- joint hip_shoulder_right_joint: limit lower=0 upper=0 effort=0 velocity=0 -> lower=-0.17453 upper=1.2217 effort=1.08 velocity=6.16; origin xyz=0.108 0.0159999999999952 0.1093 rpy=1.5707963267949 0 3.14159265358979 -> xyz=0.108 0.016 0.1093 rpy=1.5708 0 3.1416
- joint knee_ankle_left_joint: limit lower=0 upper=0 effort=0 velocity=0 -> lower=-0.34907 upper=0.69813 effort=1.08 velocity=6.16
- joint knee_ankle_right_joint: limit lower=0 upper=0 effort=0 velocity=0 -> lower=-0.69813 upper=0.34907 effort=1.08 velocity=6.16
- joint knee_knee_left_link: limit lower=0 upper=0 effort=0 velocity=0 -> lower=-1.2217 upper=1.2217 effort=1.08 velocity=6.16; origin xyz=0.0214999999999998 -0.0570000000000001 -0.0179999999999996 rpy=0 1.5707963267949 0 -> xyz=0.0215 -0.057 -0.018 rpy=0 1.5708 0
- joint shoulder_elbow_left_joint: axis 0 0 -1 -> 0 0.93969 -0.34202; limit lower=0 upper=0 effort=0 velocity=0 -> lower=-1.3963 upper=1.3963 effort=1.08 velocity=6.16; origin xyz=0 -0.0600000000000008 0 rpy=0 0 0 -> xyz=0 -0.020521 -0.056382 rpy=0 0 0
- joint shoulder_elbow_right_joint: limit lower=0 upper=0 effort=0 velocity=0 -> lower=-1.3963 upper=1.3963 effort=1.08 velocity=6.16; origin xyz=0 -0.0599999999999999 0.00350000000000003 rpy=0 0 0 -> xyz=0.051962 -0.033622 0.029672 rpy=0 0 0
- joint shoulder_shoulder_left_joint: axis 0 0 -1 -> 0 0.93969 -0.34202; limit lower=0 upper=0 effort=0 velocity=0 -> lower=-1.0472 upper=1.0472 effort=1.08 velocity=6.16; origin xyz=0.0105000000000001 -0.0205 0.0309 rpy=0 1.5707963267949 0 -> xyz=-0.015672 -0.016878 0.0309 rpy=0 1.5708 0
- joint shoulder_shoulder_right_joint: axis 0 0 -1 -> 0 0.93969 -0.34202; limit lower=0 upper=0 effort=0 velocity=0 -> lower=-1.0472 upper=1.0472 effort=1.08 velocity=6.16; origin xyz=0.0105000000000001 -0.0205000000000001 -0.0274 rpy=0 1.5707963267949 0 -> xyz=-0.015672 -0.016878 -0.0274 rpy=0 1.5708 0

Commit message: fix cad

File: Hardware/CAD/Robot/urdf/robot_humanoid/urdf/robot_humanoid.urdf (robot description, URDF)
Before this commit: robot robot_humanoid, 19 links, 18 joints
Links:
- link ankle_ankle_right_link: mass 0.085921 -> 0.0859210745449871
- link base_hip_left_link: mass 0.054051 -> 0.054051364576062
- link base_hip_middle_link: mass 0 -> 0.322024415361419
- link base_hip_right_link: mass 0.054051 -> 0.054051364576062
- link base_link: mass 0.050567 -> 0.0505669356625173
- link hip_head_link: mass 0.11435 -> 0.114347135302489
- link hip_hip_left_link: mass 0.078286 -> 0.0782857304964655
- link hip_hip_right_link: mass 0.078286 -> 0.0782857304964656
- link hip_knee_left_link: mass 0.076362 -> 0.0763616529215024
- link hip_knee_right_link: mass 0.076362 -> 0.0763616529215023
- link hip_shoulder_left_link: mass 0.054051 -> 0.054051364576062
- link hip_shoulder_right_link: mass 0.054051 -> 0.054051364576062
- link knee_ankle_left_link: mass 0.029852 -> 0.0298519989099933
- link knee_ankle_right_link: mass 0.024903 -> 0.0249034054429907
- link knee_knee_left_link: mass 0.085005 -> 0.0850053645760622
- link shoulder_elbow_left_link: mass 0.094735 -> 0.0947347359064562
- link shoulder_elbow_right_link: mass 0.094683 -> 0.09468264272445
- link shoulder_shoulder_left_link: mass 0.079491 -> 0.0794907034391992
- link shoulder_shoulder_right_link: mass 0.079491 -> 0.0794907034391992
Joints:
- joint base_hip_left_joint: limit lower=-0.69813 upper=0.17453 effort=1.08 velocity=6.16 -> lower=-0.17453 upper=0.69813 effort=1.08 velocity=6.16
- joint shoulder_elbow_left_joint: axis 0 0.93969 -0.34202 -> 0 0 -1; origin xyz=0 -0.020521 -0.056382 rpy=0 0 0 -> xyz=0 -0.063622 0.026172 rpy=0 0 0
- joint shoulder_elbow_right_joint: origin xyz=0.051962 -0.033622 0.029672 rpy=0 0 0 -> xyz=0 -0.063622 0.026172 rpy=0 0 0
- joint shoulder_shoulder_left_joint: axis 0 0.93969 -0.34202 -> 0 0 -1
- joint shoulder_shoulder_right_joint: axis 0 0.93969 -0.34202 -> 0 0 -1
