Commit message: fix uvc

File: Software/Ros2_WS/install/ros2_pkg/share/ros2_pkg/urdf/humanoid_physics.xacro (robot description, xacro)
@@ -1,8 +1,8 @@
 <?xml version="1.0"?>
 <robot xmlns:xacro="http://www.ros.org/wiki/xacro">
-  <xacro:property name="petg_mu1" value="1.2" />
-  <xacro:property name="petg_mu2" value="0.8" />
+  <xacro:property name="petg_mu1" value="1.5" />
+  <xacro:property name="petg_mu2" value="1.0" />
   <xacro:property name="petg_kp" value="1000000.0" />
-  <xacro:property name="petg_kd" value="50.0" />
+  <xacro:property name="petg_kd" value="100.0" />
   <xacro:macro name="setup_link" params="link_name">
     <gazebo reference="${link_name}">
@@ -11,12 +11,4 @@
       <kp>${petg_kp}</kp>
       <kd>${petg_kd}</kd>
-      <min_depth>0.001</min_depth>
-      <max_vel>0.1</max_vel>
-      <visual>
-        <material>
-          <diffuse>0.8 0.6 0.1 1.0</diffuse>
-          <ambient>0.8 0.6 0.1 1.0</ambient>
-        </material>
-      </visual>
     </gazebo>
   </xacro:macro>
@@ -26,17 +18,14 @@
         filename="gz-sim-joint-state-publisher-system"
         name="gz::sim::systems::JointStatePublisher">
-        <update_rate>100</update_rate>
+        <update_rate>50</update_rate>
       </plugin>
       <plugin
-        filename="gz-sim-joint-position-controller-system"
-        name="gz::sim::systems::JointPositionController">
+        filename="gz-sim-joint-trajectory-controller-system"
+        name="gz::sim::systems::JointTrajectoryController">
+        <topic>/model/humanoid_robot/joint_trajectory</topic>
       </plugin>
-      <plugin
-        filename="gz-sim-imu-system"
-        name="gz::sim::systems::Imu">
+      <plugin filename="gz-sim-imu-system" name="gz::sim::systems::Imu">
       </plugin>
-      <plugin
-        filename="gz-sim-scene-broadcaster-system"
-        name="gz::sim::systems::SceneBroadcaster">
+      <plugin filename="gz-sim-scene-broadcaster-system" name="gz::sim::systems::SceneBroadcaster">
       </plugin>
     </gazebo>

File: Software/Ros2_WS/install/ros2_pkg/share/ros2_pkg/urdf/main.xacro (robot description, xacro)
@@ -1,4 +1,10 @@
 <?xml version="1.0"?>
 <robot name="robot_humanoid" xmlns:xacro="http://www.ros.org/wiki/xacro">
+  <link name="world_root"/>
+  <joint name="world_root_joint" type="fixed">
+    <parent link="world_root"/>
+    <child link="base_link"/>
+    <origin xyz="0 0 0" rpy="0 0 0"/>
+  </joint>
   <xacro:include filename="$(find ros2_pkg)/urdf/urdf/Robot.urdf" />
   <xacro:include filename="$(find ros2_pkg)/urdf/humanoid_physics.xacro" />
@@ -16,10 +22,4 @@
   <xacro:setup_link link_name="knee_ankle_right_link" />
   <xacro:setup_link link_name="ankle_ankle_right_link" />
-  <xacro:setup_link link_name="hip_shoulder_left_link" />
-  <xacro:setup_link link_name="shoulder_shoulder_left_link" />
-  <xacro:setup_link link_name="shoulder_elbow_left_link" />
-  <xacro:setup_link link_name="hip_shoulder_right_link" />
-  <xacro:setup_link link_name="shoulder_shoulder_right_link" />
-  <xacro:setup_link link_name="shoulder_elbow_right_link" />
   <gazebo reference="base_link">
     <sensor name="imu_sensor" type="imu">
@@ -31,12 +31,9 @@
   </gazebo>
   <xacro:robot_brain />
-  <xacro:macro name="joint_dynamics" params="joint_name">
-    <gazebo reference="${joint_name}">
-      <implicitSpringDamper>true</implicitSpringDamper>
-    </gazebo>
-  </xacro:macro>
-  <xacro:joint_dynamics joint_name="hip_knee_left_joint" />
-  <xacro:joint_dynamics joint_name="hip_knee_right_joint" />
-  <xacro:joint_dynamics joint_name="knee_ankle_left_joint" />
-  <xacro:joint_dynamics joint_name="knee_ankle_right_joint" />
+  <xacro:setup_joint joint_name="hip_hip_left_joint" />
+  <xacro:setup_joint joint_name="hip_knee_left_joint" />
+  <xacro:setup_joint joint_name="knee_ankle_left_joint" />
+  <xacro:setup_joint joint_name="hip_hip_right_joint" />
+  <xacro:setup_joint joint_name="hip_knee_right_joint" />
+  <xacro:setup_joint joint_name="knee_ankle_right_joint" />
 </robot>

Commit message: fix uvc and urdf

File: Software/Ros2_WS/install/ros2_pkg/share/ros2_pkg/urdf/humanoid_physics.xacro (robot description, xacro)
@@ -1,81 +1 @@
-<?xml version="1.0"?>
-<robot xmlns:xacro="http://www.ros.org/wiki/xacro">
-  <xacro:property name="petg_mu" value="0.7" />
-  <xacro:property name="petg_kp" value="100000.0" />
-  <xacro:property name="petg_kd" value="1.0" />
-  <xacro:macro name="setup_link" params="link_name">
-    <gazebo reference="${link_name}">
-      <mu1>${petg_mu}</mu1>
-      <mu2>${petg_mu}</mu2>
-      <kp>${petg_kp}</kp>
-      <kd>${petg_kd}</kd>
-    </gazebo>
-  </xacro:macro>
-  <xacro:macro name="setup_joint" params="joint_name">
-    <gazebo reference="${joint_name}">
-      <implicitSpringDamper>true</implicitSpringDamper>
-      <springStiffness>15.0</springStiffness>
-      <springReference>0.0</springReference>
-      <friction>1.5</friction>
-      <damping>1.0</damping>
-    </gazebo>
-  </xacro:macro>
-  <xacro:macro name="make_controller" params="joint_name p d">
-    <gazebo>
-      <plugin filename="gz-sim-joint-position-controller-system"
-              name="gz::sim::systems::JointPositionController">
-        <joint_name>${joint_name}</joint_name>
-        <topic>/model/humanoid_robot/joint/${joint_name}/cmd_pos</topic>
-        <p_gain>${p}</p_gain>
-        <i_gain>0.1</i_gain>
-        <d_gain>${d}</d_gain>
-        <i_max>10</i_max>
-        <i_min>-10</i_min>
-        <cmd_max>200.0</cmd_max>
-        <cmd_min>-200.0</cmd_min>
-      </plugin>
-    </gazebo>
-  </xacro:macro>
-  <xacro:macro name="robot_brain">
-    <gazebo>
-      <plugin filename="gz-sim-joint-state-publisher-system" name="gz::sim::systems::JointStatePublisher">
-        <update_rate>500</update_rate>
-      </plugin>
-      <plugin filename="gz-sim-imu-system" name="gz::sim::systems::Imu"></plugin>
-    </gazebo>
-    <xacro:setup_joint joint_name="base_hip_left_joint"/>
-    <xacro:setup_joint joint_name="hip_hip_left_joint"/>
-    <xacro:setup_joint joint_name="hip_knee_left_joint"/>
-    <xacro:setup_joint joint_name="knee_ankle_left_joint"/>
-    <xacro:setup_joint joint_name="ankle_ankle_left_joint"/>
-    <xacro:make_controller joint_name="base_hip_left_joint"    p="5000" d="100"/>
-    <xacro:make_controller joint_name="hip_hip_left_joint"     p="5000" d="100"/>
-    <xacro:make_controller joint_name="hip_knee_left_joint"    p="8000" d="200"/>
-    <xacro:make_controller joint_name="knee_ankle_left_joint"  p="8000" d="200"/>
-    <xacro:make_controller joint_name="ankle_ankle_left_joint" p="5000" d="100"/>
-    <xacro:setup_joint joint_name="base_hip_right_joint"/>
-    <xacro:setup_joint joint_name="hip_hip_right_joint"/>
-    <xacro:setup_joint joint_name="hip_knee_right_joint"/>
-    <xacro:setup_joint joint_name="knee_ankle_right_joint"/>
-    <xacro:setup_joint joint_name="ankle_ankle_right_joint"/>
-    <xacro:make_controller joint_name="base_hip_right_joint"    p="5000" d="100"/>
-    <xacro:make_controller joint_name="hip_hip_right_joint"     p="5000" d="100"/>
-    <xacro:make_controller joint_name="hip_knee_right_joint"    p="8000" d="200"/>
-    <xacro:make_controller joint_name="knee_ankle_right_joint"  p="8000" d="200"/>
-    <xacro:make_controller joint_name="ankle_ankle_right_joint" p="5000" d="100"/>
-    <xacro:setup_joint joint_name="base_hip_middle_joint"/>
-    <xacro:make_controller joint_name="base_hip_middle_joint"   p="5000" d="100"/>
-    <xacro:setup_joint joint_name="hip_shoulder_left_joint"/>
-    <xacro:setup_joint joint_name="shoulder_shoulder_left_joint"/>
-    <xacro:setup_joint joint_name="shoulder_elbow_left_joint"/>
-    <xacro:make_controller joint_name="hip_shoulder_left_joint"      p="1500" d="50"/>
-    <xacro:make_controller joint_name="shoulder_shoulder_left_joint" p="1500" d="50"/>
-    <xacro:make_controller joint_name="shoulder_elbow_left_joint"    p="1500" d="50"/>
-    <xacro:setup_joint joint_name="hip_shoulder_right_joint"/>
-    <xacro:setup_joint joint_name="shoulder_shoulder_right_joint"/>
-    <xacro:setup_joint joint_name="shoulder_elbow_right_joint"/>
-    <xacro:make_controller joint_name="hip_shoulder_right_joint"      p="1500" d="50"/>
-    <xacro:make_controller joint_name="shoulder_shoulder_right_joint" p="1500" d="50"/>
-    <xacro:make_controller joint_name="shoulder_elbow_right_joint"    p="1500" d="50"/>
-  </xacro:macro>
-</robot>
+/home/du/Desktop/NCKH_2026/Software/Ros2_WS/src/ros2_pkg/urdf/humanoid_physics.xacro

File: Software/Ros2_WS/install/ros2_pkg/share/ros2_pkg/urdf/main.xacro (robot description, xacro)
@@ -1,34 +1 @@
-<?xml version="1.0"?>
-<robot name="robot_humanoid" xmlns:xacro="http://www.ros.org/wiki/xacro">
-  <xacro:include filename="$(find ros2_pkg)/urdf/urdf/Robot.urdf" />
-  <xacro:include filename="$(find ros2_pkg)/urdf/humanoid_physics.xacro" />
-  <xacro:setup_link link_name="base_link" />
-  <xacro:setup_link link_name="base_hip_middle_link" />
-  <xacro:setup_link link_name="hip_head_link" />
-  <xacro:setup_link link_name="base_hip_left_link" />
-  <xacro:setup_link link_name="hip_hip_left_link" />
-  <xacro:setup_link link_name="hip_knee_left_link" />
-  <xacro:setup_link link_name="knee_ankle_left_link" />
-  <xacro:setup_link link_name="ankle_ankle_left_link" />
-  <xacro:setup_link link_name="base_hip_right_link" />
-  <xacro:setup_link link_name="hip_hip_right_link" />
-  <xacro:setup_link link_name="hip_knee_right_link" />
-  <xacro:setup_link link_name="knee_ankle_right_link" />
-  <xacro:setup_link link_name="ankle_ankle_right_link" />
-  <xacro:setup_link link_name="hip_shoulder_left_link" />
-  <xacro:setup_link link_name="shoulder_shoulder_left_link" />
-  <xacro:setup_link link_name="shoulder_elbow_left_link" />
-  <xacro:setup_link link_name="hip_shoulder_right_link" />
-  <xacro:setup_link link_name="shoulder_shoulder_right_link" />
-  <xacro:setup_link link_name="shoulder_elbow_right_link" />
-  <gazebo reference="base_hip_middle_link">
-    <sensor name="imu_sensor" type="imu">
-      <always_on>1</always_on>
-      <update_rate>500</update_rate>
-      <visualize>true</visualize>
-      <topic>imu</topic>
-      <pose>0 0 0 0 0 0</pose>
-    </sensor>
-  </gazebo>
-  <xacro:robot_brain />
-</robot>
+/home/du/Desktop/NCKH_2026/Software/Ros2_WS/src/ros2_pkg/urdf/main.xacro

File: Software/Ros2_WS/src/ros2_pkg/urdf/humanoid_physics.xacro (robot description, xacro)
@@ -1,5 +1,5 @@
 <?xml version="1.0"?>
 <robot xmlns:xacro="http://www.ros.org/wiki/xacro">
-  <xacro:property name="petg_mu" value="0.7" />
+  <xacro:property name="petg_mu" value="0.85" />
   <xacro:property name="petg_kp" value="100000.0" />
   <xacro:property name="petg_kd" value="1.0" />
@@ -15,5 +15,5 @@
     <gazebo reference="${joint_name}">
       <implicitSpringDamper>true</implicitSpringDamper>
-      <springStiffness>15.0</springStiffness>
+      <springStiffness>0.0</springStiffness>
       <springReference>0.0</springReference>
       <friction>1.5</friction>
@@ -49,9 +49,9 @@
     <xacro:setup_joint joint_name="knee_ankle_left_joint"/>
     <xacro:setup_joint joint_name="ankle_ankle_left_joint"/>
-    <xacro:make_controller joint_name="base_hip_left_joint"    p="5000" d="100"/>
-    <xacro:make_controller joint_name="hip_hip_left_joint"     p="5000" d="100"/>
-    <xacro:make_controller joint_name="hip_knee_left_joint"    p="8000" d="200"/>
-    <xacro:make_controller joint_name="knee_ankle_left_joint"  p="8000" d="200"/>
-    <xacro:make_controller joint_name="ankle_ankle_left_joint" p="5000" d="100"/>
+    <xacro:make_controller joint_name="base_hip_left_joint"    p="800" d="10"/>
+    <xacro:make_controller joint_name="hip_hip_left_joint"     p="800" d="10"/>
+    <xacro:make_controller joint_name="hip_knee_left_joint"    p="800" d="10"/>
+    <xacro:make_controller joint_name="knee_ankle_left_joint"  p="800" d="10"/>
+    <xacro:make_controller joint_name="ankle_ankle_left_joint" p="800" d="10"/>
     <xacro:setup_joint joint_name="base_hip_right_joint"/>
     <xacro:setup_joint joint_name="hip_hip_right_joint"/>
@@ -59,23 +59,23 @@
     <xacro:setup_joint joint_name="knee_ankle_right_joint"/>
     <xacro:setup_joint joint_name="ankle_ankle_right_joint"/>
-    <xacro:make_controller joint_name="base_hip_right_joint"    p="5000" d="100"/>
-    <xacro:make_controller joint_name="hip_hip_right_joint"     p="5000" d="100"/>
-    <xacro:make_controller joint_name="hip_knee_right_joint"    p="8000" d="200"/>
-    <xacro:make_controller joint_name="knee_ankle_right_joint"  p="8000" d="200"/>
-    <xacro:make_controller joint_name="ankle_ankle_right_joint" p="5000" d="100"/>
+    <xacro:make_controller joint_name="base_hip_right_joint"    p="800" d="10"/>
+    <xacro:make_controller joint_name="hip_hip_right_joint"     p="800" d="10"/>
+    <xacro:make_controller joint_name="hip_knee_right_joint"    p="800" d="10"/>
+    <xacro:make_controller joint_name="knee_ankle_right_joint"  p="800" d="10"/>
+    <xacro:make_controller joint_name="ankle_ankle_right_joint" p="800" d="10"/>
     <xacro:setup_joint joint_name="base_hip_middle_joint"/>
-    <xacro:make_controller joint_name="base_hip_middle_joint"   p="5000" d="100"/>
+    <xacro:make_controller joint_name="base_hip_middle_joint"   p="800" d="10"/>
     <xacro:setup_joint joint_name="hip_shoulder_left_joint"/>
     <xacro:setup_joint joint_name="shoulder_shoulder_left_joint"/>
     <xacro:setup_joint joint_name="shoulder_elbow_left_joint"/>
-    <xacro:make_controller joint_name="hip_shoulder_left_joint"      p="1500" d="50"/>
-    <xacro:make_controller joint_name="shoulder_shoulder_left_joint" p="1500" d="50"/>
-    <xacro:make_controller joint_name="shoulder_elbow_left_joint"    p="1500" d="50"/>
+    <xacro:make_controller joint_name="hip_shoulder_left_joint"      p="800" d="10"/>
+    <xacro:make_controller joint_name="shoulder_shoulder_left_joint" p="800" d="10"/>
+    <xacro:make_controller joint_name="shoulder_elbow_left_joint"    p="800" d="10"/>
     <xacro:setup_joint joint_name="hip_shoulder_right_joint"/>
     <xacro:setup_joint joint_name="shoulder_shoulder_right_joint"/>
     <xacro:setup_joint joint_name="shoulder_elbow_right_joint"/>
-    <xacro:make_controller joint_name="hip_shoulder_right_joint"      p="1500" d="50"/>
-    <xacro:make_controller joint_name="shoulder_shoulder_right_joint" p="1500" d="50"/>
-    <xacro:make_controller joint_name="shoulder_elbow_right_joint"    p="1500" d="50"/>
+    <xacro:make_controller joint_name="hip_shoulder_right_joint"      p="800" d="10"/>
+    <xacro:make_controller joint_name="shoulder_shoulder_right_joint" p="800" d="10"/>
+    <xacro:make_controller joint_name="shoulder_elbow_right_joint"    p="800" d="10"/>
   </xacro:macro>
 </robot>

File: Software/Ros2_WS/src/ros2_pkg/urdf/main.xacro (robot description, xacro)
@@ -24,5 +24,5 @@
   <gazebo reference="base_hip_middle_link">
     <sensor name="imu_sensor" type="imu">
-      <always_on>1</always_on>
+      <always_on>0</always_on>
       <update_rate>500</update_rate>
       <visualize>true</visualize>

File: Software/Ros2_WS/src/ros2_pkg/urdf/urdf/Robot.urdf (robot description, URDF)
Before this commit: robot Robot, 19 links, 18 joints
Joints:
- joint hip_hip_left_joint: limit lower=-0.5236 upper=0.69813 effort=0.8 velocity=6.16 -> lower=-0.8 upper=0.69813 effort=0.8 velocity=6.16
- joint hip_hip_right_joint: limit lower=-0.69813 upper=0.5236 effort=0.8 velocity=6.16 -> lower=-0.69813 upper=0.8 effort=0.8 velocity=6.16
- joint knee_ankle_left_joint: limit lower=-0.34907 upper=0.69813 effort=0.8 velocity=6.16 -> lower=-0.8 upper=0.8 effort=0.8 velocity=6.16
- joint knee_ankle_right_joint: limit lower=-0.69813 upper=0.34907 effort=0.8 velocity=6.16 -> lower=-0.8 upper=0.8 effort=0.8 velocity=6.16

Commit message: fix uvc

File: Software/Ros2_WS/install/ros2_pkg/share/ros2_pkg/urdf/humanoid_physics.xacro (robot description, xacro)
@@ -1 +1,81 @@
-/home/dat/NCKH_2026/Software/Ros2_WS/src/ros2_pkg/urdf/humanoid_physics.xacro
+<?xml version="1.0"?>
+<robot xmlns:xacro="http://www.ros.org/wiki/xacro">
+  <xacro:property name="petg_mu" value="0.85" />
+  <xacro:property name="petg_kp" value="100000.0" />
+  <xacro:property name="petg_kd" value="1.0" />
+  <xacro:macro name="setup_link" params="link_name">
+    <gazebo reference="${link_name}">
+      <mu1>${petg_mu}</mu1>
+      <mu2>${petg_mu}</mu2>
+      <kp>${petg_kp}</kp>
+      <kd>${petg_kd}</kd>
+    </gazebo>
+  </xacro:macro>
+  <xacro:macro name="setup_joint" params="joint_name">
+    <gazebo reference="${joint_name}">
+      <implicitSpringDamper>true</implicitSpringDamper>
+      <springStiffness>5.0</springStiffness>
+      <springReference>0.0</springReference>
+      <friction>1.5</friction>
+      <damping>1.0</damping>
+    </gazebo>
+  </xacro:macro>
+  <xacro:macro name="make_controller" params="joint_name p d">
+    <gazebo>
+      <plugin filename="gz-sim-joint-position-controller-system"
+              name="gz::sim::systems::JointPositionController">
+        <joint_name>${joint_name}</joint_name>
+        <topic>/model/humanoid_robot/joint/${joint_name}/cmd_pos</topic>
+        <p_gain>${p}</p_gain>
+        <i_gain>0.5</i_gain>
+        <d_gain>${d}</d_gain>
+        <i_max>10</i_max>
+        <i_min>-10</i_min>
+        <cmd_max>200.0</cmd_max>
+        <cmd_min>-200.0</cmd_min>
+      </plugin>
+    </gazebo>
+  </xacro:macro>
+  <xacro:macro name="robot_brain">
+    <gazebo>
+      <plugin filename="gz-sim-joint-state-publisher-system" name="gz::sim::systems::JointStatePublisher">
+        <update_rate>100</update_rate>
+      </plugin>
+      <plugin filename="gz-sim-imu-system" name="gz::sim::systems::Imu"></plugin>
+    </gazebo>
+    <xacro:setup_joint joint_name="base_hip_left_joint"/>
+    <xacro:setup_joint joint_name="hip_hip_left_joint"/>
+    <xacro:setup_joint joint_name="hip_knee_left_joint"/>
+    <xacro:setup_joint joint_name="knee_ankle_left_joint"/>
+    <xacro:setup_joint joint_name="ankle_ankle_left_joint"/>
+    <xacro:make_controller joint_name="base_hip_left_joint"    p="8000" d="100"/>
+    <xacro:make_controller joint_name="hip_hip_left_joint"     p="8000" d="100"/>
+    <xacro:make_controller joint_name="hip_knee_left_joint"    p="8000" d="100"/>
+    <xacro:make_controller joint_name="knee_ankle_left_joint"  p="8000" d="100"/>
+    <xacro:make_controller joint_name="ankle_ankle_left_joint" p="8000" d="100"/>
+    <xacro:setup_joint joint_name="base_hip_right_joint"/>
+    <xacro:setup_joint joint_name="hip_hip_right_joint"/>
+    <xacro:setup_joint joint_name="hip_knee_right_joint"/>
+    <xacro:setup_joint joint_name="knee_ankle_right_joint"/>
+    <xacro:setup_joint joint_name="ankle_ankle_right_joint"/>
+    <xacro:make_controller joint_name="base_hip_right_joint"    p="8000" d="100"/>
+    <xacro:make_controller joint_name="hip_hip_right_joint"     p="8000" d="100"/>
+    <xacro:make_controller joint_name="hip_knee_right_joint"    p="8000" d="100"/>
+    <xacro:make_controller joint_name="knee_ankle_right_joint"  p="8000" d="100"/>
+    <xacro:make_controller joint_name="ankle_ankle_right_joint" p="8000" d="100"/>
+    <xacro:setup_joint joint_name="base_hip_middle_joint"/>
+    <xacro:make_controller joint_name="base_hip_middle_joint"   p="8000" d="100"/>
+    <xacro:setup_joint joint_name="hip_shoulder_left_joint"/>
+    <xacro:setup_joint joint_name="shoulder_shoulder_left_joint"/>
+    <xacro:setup_joint joint_name="shoulder_elbow_left_joint"/>
+    <xacro:make_controller joint_name="hip_shoulder_left_joint"      p="8000" d="100"/>
+    <xacro:make_controller joint_name="shoulder_shoulder_left_joint" p="8000" d="100"/>
+    <xacro:make_controller joint_name="shoulder_elbow_left_joint"    p="8000" d="100"/>
+    <xacro:setup_joint joint_name="hip_shoulder_right_joint"/>
+    <xacro:setup_joint joint_name="shoulder_shoulder_right_joint"/>
+    <xacro:setup_joint joint_name="shoulder_elbow_right_joint"/>
+    <xacro:make_controller joint_name="hip_shoulder_right_joint"      p="8000" d="100"/>
+    <xacro:make_controller joint_name="shoulder_shoulder_right_joint" p="8000" d="100"/>
+    <xacro:make_controller joint_name="shoulder_elbow_right_joint"    p="8000" d="100"/>
+  </xacro:macro>
+</robot>

File: Software/Ros2_WS/install/ros2_pkg/share/ros2_pkg/urdf/main.xacro (robot description, xacro)
@@ -1 +1,34 @@
-/home/dat/NCKH_2026/Software/Ros2_WS/src/ros2_pkg/urdf/main.xacro
+<?xml version="1.0"?>
+<robot name="robot_humanoid" xmlns:xacro="http://www.ros.org/wiki/xacro">
+  <xacro:include filename="$(find ros2_pkg)/urdf/urdf/Robot.urdf" />
+  <xacro:include filename="$(find ros2_pkg)/urdf/humanoid_physics.xacro" />
+  <xacro:setup_link link_name="base_link" />
+  <xacro:setup_link link_name="base_hip_middle_link" />
+  <xacro:setup_link link_name="hip_head_link" />
+  <xacro:setup_link link_name="base_hip_left_link" />
+  <xacro:setup_link link_name="hip_hip_left_link" />
+  <xacro:setup_link link_name="hip_knee_left_link" />
+  <xacro:setup_link link_name="knee_ankle_left_link" />
+  <xacro:setup_link link_name="ankle_ankle_left_link" />
+  <xacro:setup_link link_name="base_hip_right_link" />
+  <xacro:setup_link link_name="hip_hip_right_link" />
+  <xacro:setup_link link_name="hip_knee_right_link" />
+  <xacro:setup_link link_name="knee_ankle_right_link" />
+  <xacro:setup_link link_name="ankle_ankle_right_link" />
+  <xacro:setup_link link_name="hip_shoulder_left_link" />
+  <xacro:setup_link link_name="shoulder_shoulder_left_link" />
+  <xacro:setup_link link_name="shoulder_elbow_left_link" />
+  <xacro:setup_link link_name="hip_shoulder_right_link" />
+  <xacro:setup_link link_name="shoulder_shoulder_right_link" />
+  <xacro:setup_link link_name="shoulder_elbow_right_link" />
+  <gazebo reference="base_hip_middle_link">
+    <sensor name="imu_sensor" type="imu">
+      <always_on>0</always_on>
+      <update_rate>100</update_rate>
+      <visualize>true</visualize>
+      <topic>imu</topic>
+      <pose>0 0 0 0 0 0</pose>
+    </sensor>
+  </gazebo>
+  <xacro:robot_brain />
+</robot>

File: Software/Ros2_WS/src/ros2_pkg/urdf/humanoid_physics.xacro (robot description, xacro)
@@ -15,5 +15,5 @@
     <gazebo reference="${joint_name}">
       <implicitSpringDamper>true</implicitSpringDamper>
-      <springStiffness>1.0</springStiffness>
+      <springStiffness>5.0</springStiffness>
       <springReference>0.0</springReference>
       <friction>1.5</friction>
