Commit message: fix ik

File: Software/Ros2_WS/install/ros2_pkg/share/ros2_pkg/urdf/humanoid_physics.xacro (robot description, xacro)
@@ -1,7 +1,7 @@
 <?xml version="1.0"?>
 <robot xmlns:xacro="http://www.ros.org/wiki/xacro">
-  <xacro:property name="petg_mu" value="0.85" />
-  <xacro:property name="petg_kp" value="100000.0" />
-  <xacro:property name="petg_kd" value="1.0" />
+  <xacro:property name="petg_mu" value="1.0" />
+  <xacro:property name="petg_kp" value="1000000.0" />
+  <xacro:property name="petg_kd" value="100.0" />
   <xacro:macro name="setup_link" params="link_name">
     <gazebo reference="${link_name}">
@@ -15,5 +15,5 @@
     <gazebo reference="${joint_name}">
       <implicitSpringDamper>true</implicitSpringDamper>
-      <springStiffness>5.0</springStiffness>
+      <springStiffness>0.0</springStiffness>
       <springReference>0.0</springReference>
       <friction>1.5</friction>

Commit message: add rl

File: Software/Ros2_WS/install/ros2_pkg/share/ros2_pkg/urdf/humanoid_physics.xacro (robot description, xacro)
@@ -1,81 +1 @@
-<?xml version="1.0"?>
-<robot xmlns:xacro="http://www.ros.org/wiki/xacro">
-  <xacro:property name="petg_mu" value="1.0" />
-  <xacro:property name="petg_kp" value="1000000.0" />
-  <xacro:property name="petg_kd" value="100.0" />
-  <xacro:macro name="setup_link" params="link_name">
-    <gazebo reference="${link_name}">
-      <mu1>${petg_mu}</mu1>
-      <mu2>${petg_mu}</mu2>
-      <kp>${petg_kp}</kp>
-      <kd>${petg_kd}</kd>
-    </gazebo>
-  </xacro:macro>
-  <xacro:macro name="setup_joint" params="joint_name">
-    <gazebo reference="${joint_name}">
-      <implicitSpringDamper>true</implicitSpringDamper>
-      <springStiffness>0.0</springStiffness>
-      <springReference>0.0</springReference>
-      <friction>1.5</friction>
-      <damping>1.0</damping>
-    </gazebo>
-  </xacro:macro>
-  <xacro:macro name="make_controller" params="joint_name p d">
-    <gazebo>
-      <plugin filename="gz-sim-joint-position-controller-system"
-              name="gz::sim::systems::JointPositionController">
-        <joint_name>${joint_name}</joint_name>
-        <topic>/model/humanoid_robot/joint/${joint_name}/cmd_pos</topic>
-        <p_gain>${p}</p_gain>
-        <i_gain>0.5</i_gain>
-        <d_gain>${d}</d_gain>
-        <i_max>10</i_max>
-        <i_min>-10</i_min>
-        <cmd_max>200.0</cmd_max>
-        <cmd_min>-200.0</cmd_min>
-      </plugin>
-    </gazebo>
-  </xacro:macro>
-  <xacro:macro name="robot_brain">
-    <gazebo>
-      <plugin filename="gz-sim-joint-state-publisher-system" name="gz::sim::systems::JointStatePublisher">
-        <update_rate>100</update_rate>
-      </plugin>
-      <plugin filename="gz-sim-imu-system" name="gz::sim::systems::Imu"></plugin>
-    </gazebo>
-    <xacro:setup_joint joint_name="base_hip_left_joint"/>
-    <xacro:setup_joint joint_name="hip_hip_left_joint"/>
-    <xacro:setup_joint joint_name="hip_knee_left_joint"/>
-    <xacro:setup_joint joint_name="knee_ankle_left_joint"/>
-    <xacro:setup_joint joint_name="ankle_ankle_left_joint"/>
-    <xacro:make_controller joint_name="base_hip_left_joint"    p="8000" d="100"/>
-    <xacro:make_controller joint_name="hip_hip_left_joint"     p="8000" d="100"/>
-    <xacro:make_controller joint_name="hip_knee_left_joint"    p="8000" d="100"/>
-    <xacro:make_controller joint_name="knee_ankle_left_joint"  p="8000" d="100"/>
-    <xacro:make_controller joint_name="ankle_ankle_left_joint" p="8000" d="100"/>
-    <xacro:setup_joint joint_name="base_hip_right_joint"/>
-    <xacro:setup_joint joint_name="hip_hip_right_joint"/>
-    <xacro:setup_joint joint_name="hip_knee_right_joint"/>
-    <xacro:setup_joint joint_name="knee_ankle_right_joint"/>
-    <xacro:setup_joint joint_name="ankle_ankle_right_joint"/>
-    <xacro:make_controller joint_name="base_hip_right_joint"    p="8000" d="100"/>
-    <xacro:make_controller joint_name="hip_hip_right_joint"     p="8000" d="100"/>
-    <xacro:make_controller joint_name="hip_knee_right_joint"    p="8000" d="100"/>
-    <xacro:make_controller joint_name="knee_ankle_right_joint"  p="8000" d="100"/>
-    <xacro:make_controller joint_name="ankle_ankle_right_joint" p="8000" d="100"/>
-    <xacro:setup_joint joint_name="base_hip_middle_joint"/>
-    <xacro:make_controller joint_name="base_hip_middle_joint"   p="8000" d="100"/>
-    <xacro:setup_joint joint_name="hip_shoulder_left_joint"/>
-    <xacro:setup_joint joint_name="shoulder_shoulder_left_joint"/>
-    <xacro:setup_joint joint_name="shoulder_elbow_left_joint"/>
-    <xacro:make_controller joint_name="hip_shoulder_left_joint"      p="8000" d="100"/>
-    <xacro:make_controller joint_name="shoulder_shoulder_left_joint" p="8000" d="100"/>
-    <xacro:make_controller joint_name="shoulder_elbow_left_joint"    p="8000" d="100"/>
-    <xacro:setup_joint joint_name="hip_shoulder_right_joint"/>
-    <xacro:setup_joint joint_name="shoulder_shoulder_right_joint"/>
-    <xacro:setup_joint joint_name="shoulder_elbow_right_joint"/>
-    <xacro:make_controller joint_name="hip_shoulder_right_joint"      p="8000" d="100"/>
-    <xacro:make_controller joint_name="shoulder_shoulder_right_joint" p="8000" d="100"/>
-    <xacro:make_controller joint_name="shoulder_elbow_right_joint"    p="8000" d="100"/>
-  </xacro:macro>
-</robot>
+/home/du/Desktop/NCKH_2026/Software/Ros2_WS/src/ros2_pkg/urdf/humanoid_physics.xacro

File: Software/Ros2_WS/install/ros2_pkg/share/ros2_pkg/urdf/main.xacro (robot description, xacro)
@@ -1,34 +1 @@
-<?xml version="1.0"?>
-<robot name="robot_humanoid" xmlns:xacro="http://www.ros.org/wiki/xacro">
-  <xacro:include filename="$(find ros2_pkg)/urdf/urdf/Robot.urdf" />
-  <xacro:include filename="$(find ros2_pkg)/urdf/humanoid_physics.xacro" />
-  <xacro:setup_link link_name="base_link" />
-  <xacro:setup_link link_name="base_hip_middle_link" />
-  <xacro:setup_link link_name="hip_head_link" />
-  <xacro:setup_link link_name="base_hip_left_link" />
-  <xacro:setup_link link_name="hip_hip_left_link" />
-  <xacro:setup_link link_name="hip_knee_left_link" />
-  <xacro:setup_link link_name="knee_ankle_left_link" />
-  <xacro:setup_link link_name="ankle_ankle_left_link" />
-  <xacro:setup_link link_name="base_hip_right_link" />
-  <xacro:setup_link link_name="hip_hip_right_link" />
-  <xacro:setup_link link_name="hip_knee_right_link" />
-  <xacro:setup_link link_name="knee_ankle_right_link" />
-  <xacro:setup_link link_name="ankle_ankle_right_link" />
-  <xacro:setup_link link_name="hip_shoulder_left_link" />
-  <xacro:setup_link link_name="shoulder_shoulder_left_link" />
-  <xacro:setup_link link_name="shoulder_elbow_left_link" />
-  <xacro:setup_link link_name="hip_shoulder_right_link" />
-  <xacro:setup_link link_name="shoulder_shoulder_right_link" />
-  <xacro:setup_link link_name="shoulder_elbow_right_link" />
-  <gazebo reference="base_hip_middle_link">
-    <sensor name="imu_sensor" type="imu">
-      <always_on>0</always_on>
-      <update_rate>100</update_rate>
-      <visualize>true</visualize>
-      <topic>imu</topic>
-      <pose>0 0 0 0 0 0</pose>
-    </sensor>
-  </gazebo>
-  <xacro:robot_brain />
-</robot>
+/home/du/Desktop/NCKH_2026/Software/Ros2_WS/src/ros2_pkg/urdf/main.xacro

Commit message: add sp

File: Software/Ros2_WS/install/ros2_pkg/share/ros2_pkg/urdf/humanoid_physics.xacro (robot description, xacro)
@@ -1 +1 @@
-/home/nckh/Desktop/NCKH_2026/Software/Ros2_WS/src/ros2_pkg/urdf/humanoid_physics.xacro
+/home/du/Desktop/NCKH_2026/Software/Ros2_WS/src/ros2_pkg/urdf/humanoid_physics.xacro

File: Software/Ros2_WS/install/ros2_pkg/share/ros2_pkg/urdf/main.xacro (robot description, xacro)
@@ -1 +1 @@
-/home/nckh/Desktop/NCKH_2026/Software/Ros2_WS/src/ros2_pkg/urdf/main.xacro
+/home/du/Desktop/NCKH_2026/Software/Ros2_WS/src/ros2_pkg/urdf/main.xacro

File: Software/Ros2_WS/install/ros2_pkg/share/ros2_pkg/urdf/main_turbo.xacro (robot description, xacro)
@@ -1 +1 @@
-/home/nckh/Desktop/NCKH_2026/Software/Ros2_WS/src/ros2_pkg/urdf/main_turbo.xacro
+/home/du/Desktop/NCKH_2026/Software/Ros2_WS/src/ros2_pkg/urdf/main_turbo.xacro

File: Software/Ros2_WS/src/ros2_pkg/urdf/humanoid_physics.xacro (robot description, xacro)
@@ -4,13 +4,13 @@
   <xacro:property name="petg_kp" value="100000.0" />
   <xacro:property name="petg_kd" value="10.0" />
-  <xacro:property name="silicone_mu" value="0.8" />
+  <xacro:property name="silicone_mu" value="0.99" />
   <xacro:property name="silicone_kp" value="40000.0" />
-  <xacro:property name="silicone_kd" value="12.0" />
+  <xacro:property name="silicone_kd" value="25.0" />
   <xacro:property name="silicone_thickness" value="0.002" />
   <xacro:macro name="setup_joint" params="joint_name">
     <gazebo reference="${joint_name}">
       <implicitSpringDamper>true</implicitSpringDamper>
-      <friction>0.2</friction>
-      <damping>0.1</damping>
+      <friction>0.1</friction>
+      <damping>0.05</damping>
     </gazebo>
   </xacro:macro>
@@ -23,5 +23,5 @@
     </gazebo>
   </xacro:macro>
-  <xacro:macro name="make_controller" params="joint_name p d">
+<xacro:macro name="make_controller" params="joint_name p d">
     <gazebo>
       <plugin filename="gz-sim-joint-position-controller-system"
@@ -30,10 +30,8 @@
         <topic>/model/humanoid_robot/joint/${joint_name}/cmd_pos</topic>
         <p_gain>${p}</p_gain>
-        <i_gain>0.01</i_gain>
-        <d_gain>${d}</d_gain>
-        <i_max>1</i_max>
-        <i_min>-1</i_min>
-        <cmd_max>2.5</cmd_max>
-        <cmd_min>-2.5</cmd_min>
+        <i_gain>0.0</i_gain> <d_gain>${d}</d_gain>
+        <cmd_max>20.0</cmd_max>
+        <cmd_min>-20.0</cmd_min>
+        <velocity_max>6.0</velocity_max>
       </plugin>
     </gazebo>

File: Software/Ros2_WS/src/ros2_pkg/urdf/main.xacro (robot description, xacro)
@@ -3,4 +3,10 @@
   <xacro:include filename="$(find ros2_pkg)/urdf/urdf/Robot.urdf" />
   <xacro:include filename="$(find ros2_pkg)/urdf/humanoid_physics.xacro" />
+  <link name="base_footprint"/>
+  <joint name="base_footprint_joint" type="fixed">
+    <parent link="base_footprint"/>
+    <child link="base_link"/>
+    <origin xyz="0 0 0" rpy="0 0 0"/>
+  </joint>
   <xacro:setup_link link_name="base_link" />
   <xacro:setup_link link_name="base_hip_middle_link" />
@@ -24,6 +30,5 @@
   <gazebo reference="base_hip_middle_link">
     <sensor name="imu_sensor" type="imu">
-      <always_on>0</always_on>
-      <update_rate>100</update_rate>
+      <always_on>1</always_on> <update_rate>100</update_rate>
       <visualize>true</visualize>
       <topic>imu</topic>
