Commit message: changed to 70D input PPO

File: Software/Ros2_WS/install/ros2_pkg/share/ros2_pkg/urdf/humanoid_physics.xacro (robot description, xacro)
@@ -1,93 +1 @@
-<?xml version="1.0"?>
-<robot xmlns:xacro="http://www.ros.org/wiki/xacro">
-  <xacro:property name="petg_mu" value="0.6" />
-  <xacro:property name="petg_kp" value="100000.0" />
-  <xacro:property name="petg_kd" value="10.0" />
-  <xacro:property name="silicone_mu" value="0.99" />
-  <xacro:property name="silicone_kp" value="40000.0" />
-  <xacro:property name="silicone_kd" value="25.0" />
-  <xacro:property name="silicone_thickness" value="0.002" />
-  <xacro:macro name="setup_joint" params="joint_name">
-    <gazebo reference="${joint_name}">
-      <implicitSpringDamper>true</implicitSpringDamper>
-      <friction>0.1</friction>
-      <damping>0.05</damping>
-    </gazebo>
-  </xacro:macro>
-  <xacro:macro name="setup_link" params="link_name">
-    <gazebo reference="${link_name}">
-      <mu1>${petg_mu}</mu1>
-      <mu2>${petg_mu}</mu2>
-      <kp>${petg_kp}</kp>
-      <kd>${petg_kd}</kd>
-    </gazebo>
-  </xacro:macro>
-<xacro:macro name="make_controller" params="joint_name p d">
-    <gazebo>
-      <plugin filename="gz-sim-joint-position-controller-system"
-              name="gz::sim::systems::JointPositionController">
-        <joint_name>${joint_name}</joint_name>
-        <topic>/model/humanoid_robot/joint/${joint_name}/cmd_pos</topic>
-        <p_gain>${p}</p_gain>
-        <i_gain>0.0</i_gain> <d_gain>${d}</d_gain>
-        <cmd_max>20.0</cmd_max>
-        <cmd_min>-20.0</cmd_min>
-        <velocity_max>6.0</velocity_max>
-      </plugin>
-    </gazebo>
-  </xacro:macro>
-  <xacro:macro name="robot_brain">
-    <gazebo>
-      <plugin filename="gz-sim-joint-state-publisher-system" name="gz::sim::systems::JointStatePublisher">
-        <update_rate>100</update_rate>
-      </plugin>
-      <plugin filename="gz-sim-imu-system" name="gz::sim::systems::Imu"></plugin>
-    </gazebo>
-    <xacro:setup_joint joint_name="base_hip_left_joint"/>
-    <xacro:make_controller joint_name="base_hip_left_joint"    p="2000" d="20"/>
-    <xacro:setup_joint joint_name="hip_hip_left_joint"/>
-    <xacro:make_controller joint_name="hip_hip_left_joint"     p="2000" d="20"/>
-    <xacro:setup_joint joint_name="hip_knee_left_joint"/>
-    <xacro:make_controller joint_name="hip_knee_left_joint"    p="2000" d="20"/>
-    <xacro:setup_joint joint_name="knee_ankle_left_joint"/>
-    <xacro:make_controller joint_name="knee_ankle_left_joint"  p="2000" d="20"/>
-    <xacro:setup_joint joint_name="ankle_ankle_left_joint"/>
-    <xacro:make_controller joint_name="ankle_ankle_left_joint" p="2000" d="20"/>
-    <gazebo reference="ankle_ankle_left_link">
-      <mu1>${silicone_mu}</mu1>
-      <mu2>${silicone_mu}</mu2>
-      <kp>${silicone_kp}</kp>
-      <kd>${silicone_kd}</kd>
-    </gazebo>
-    <xacro:setup_joint joint_name="base_hip_right_joint"/>
-    <xacro:make_controller joint_name="base_hip_right_joint"    p="2000" d="20"/>
-    <xacro:setup_joint joint_name="hip_hip_right_joint"/>
-    <xacro:make_controller joint_name="hip_hip_right_joint"     p="2000" d="20"/>
-    <xacro:setup_joint joint_name="hip_knee_right_joint"/>
-    <xacro:make_controller joint_name="hip_knee_right_joint"    p="2000" d="20"/>
-    <xacro:setup_joint joint_name="knee_ankle_right_joint"/>
-    <xacro:make_controller joint_name="knee_ankle_right_joint"  p="2000" d="20"/>
-    <xacro:setup_joint joint_name="ankle_ankle_right_joint"/>
-    <xacro:make_controller joint_name="ankle_ankle_right_joint" p="2000" d="20"/>
-    <gazebo reference="ankle_ankle_right_link">
-      <mu1>${silicone_mu}</mu1>
-      <mu2>${silicone_mu}</mu2>
-      <kp>${silicone_kp}</kp>
-      <kd>${silicone_kd}</kd>
-    </gazebo>
-    <xacro:setup_joint joint_name="base_hip_middle_joint"/>
-    <xacro:make_controller joint_name="base_hip_middle_joint"   p="300" d="5"/>
-    <xacro:setup_joint joint_name="hip_shoulder_left_joint"/>
-    <xacro:make_controller joint_name="hip_shoulder_left_joint"      p="200" d="5"/>
-    <xacro:setup_joint joint_name="shoulder_shoulder_left_joint"/>
-    <xacro:make_controller joint_name="shoulder_shoulder_left_joint" p="200" d="5"/>
-    <xacro:setup_joint joint_name="shoulder_elbow_left_joint"/>
-    <xacro:make_controller joint_name="shoulder_elbow_left_joint"    p="200" d="5"/>
-    <xacro:setup_joint joint_name="hip_shoulder_right_joint"/>
-    <xacro:make_controller joint_name="hip_shoulder_right_joint"      p="200" d="5"/>
-    <xacro:setup_joint joint_name="shoulder_shoulder_right_joint"/>
-    <xacro:make_controller joint_name="shoulder_shoulder_right_joint" p="200" d="5"/>
-    <xacro:setup_joint joint_name="shoulder_elbow_right_joint"/>
-    <xacro:make_controller joint_name="shoulder_elbow_right_joint"    p="200" d="5"/>
-  </xacro:macro>
-</robot>
+/home/du/Desktop/NCKH_2026/Software/Ros2_WS/src/ros2_pkg/urdf/humanoid_physics.xacro

File: Software/Ros2_WS/install/ros2_pkg/share/ros2_pkg/urdf/main.xacro (robot description, xacro)
@@ -1,39 +1 @@
-<?xml version="1.0"?>
-<robot name="robot_humanoid" xmlns:xacro="http://www.ros.org/wiki/xacro">
-  <xacro:include filename="$(find ros2_pkg)/urdf/urdf/Robot.urdf" />
-  <xacro:include filename="$(find ros2_pkg)/urdf/humanoid_physics.xacro" />
-  <link name="base_footprint"/>
-  <joint name="base_footprint_joint" type="fixed">
-    <parent link="base_footprint"/>
-    <child link="base_link"/>
-    <origin xyz="0 0 0" rpy="0 0 0"/>
-  </joint>
-  <xacro:setup_link link_name="base_link" />
-  <xacro:setup_link link_name="base_hip_middle_link" />
-  <xacro:setup_link link_name="hip_head_link" />
-  <xacro:setup_link link_name="base_hip_left_link" />
-  <xacro:setup_link link_name="hip_hip_left_link" />
-  <xacro:setup_link link_name="hip_knee_left_link" />
-  <xacro:setup_link link_name="knee_ankle_left_link" />
-  <xacro:setup_link link_name="ankle_ankle_left_link" />
-  <xacro:setup_link link_name="base_hip_right_link" />
-  <xacro:setup_link link_name="hip_hip_right_link" />
-  <xacro:setup_link link_name="hip_knee_right_link" />
-  <xacro:setup_link link_name="knee_ankle_right_link" />
-  <xacro:setup_link link_name="ankle_ankle_right_link" />
-  <xacro:setup_link link_name="hip_shoulder_left_link" />
-  <xacro:setup_link link_name="shoulder_shoulder_left_link" />
-  <xacro:setup_link link_name="shoulder_elbow_left_link" />
-  <xacro:setup_link link_name="hip_shoulder_right_link" />
-  <xacro:setup_link link_name="shoulder_shoulder_right_link" />
-  <xacro:setup_link link_name="shoulder_elbow_right_link" />
-  <gazebo reference="base_hip_middle_link">
-    <sensor name="imu_sensor" type="imu">
-      <always_on>1</always_on> <update_rate>100</update_rate>
-      <visualize>true</visualize>
-      <topic>imu</topic>
-      <pose>0 0 0 0 0 0</pose>
-    </sensor>
-  </gazebo>
-  <xacro:robot_brain />
-</robot>
+/home/du/Desktop/NCKH_2026/Software/Ros2_WS/src/ros2_pkg/urdf/main.xacro

File: Software/Ros2_WS/install/ros2_pkg/share/ros2_pkg/urdf/main_turbo.xacro (robot description, xacro)
@@ -1,263 +1 @@
-<?xml version="1.0"?>
-<robot name="robot_humanoid" xmlns:xacro="http://www.ros.org/wiki/xacro">
-  <xacro:include filename="$(find ros2_pkg)/urdf/humanoid_physics.xacro" />
-  <xacro:macro name="turbo_link" params="name mesh_file mass ixx ixy ixz iyy iyz izz size xyz rpy mu_val:=1.0">
-    <link name="${name}">
-      <inertial>
-        <origin xyz="0 0 0" rpy="0 0 0" />
-        <mass value="${mass}" />
-        <inertia ixx="${ixx}" ixy="${ixy}" ixz="${ixz}" iyy="${iyy}" iyz="${iyz}" izz="${izz}" />
-      </inertial>
-      <visual>
-        <origin xyz="0 0 0" rpy="0 0 0" />
-        <geometry>
-          <mesh filename="package://ros2_pkg/urdf/meshes/${mesh_file}" />
-        </geometry>
-        <material name="">
-          <color rgba="0.7 0.7 0.7 1" />
-        </material>
-      </visual>
-      <collision>
-        <origin xyz="${xyz}" rpy="${rpy}" />
-        <geometry>
-          <box size="${size}" />
-        </geometry>
-        <surface>
-          <friction>
-            <ode>
-              <mu>${mu_val}</mu>
-              <mu2>${mu_val}</mu2>
-              <kp>${petg_kp}</kp> <kd>${petg_kd}</kd>
-            </ode>
-          </friction>
-        </surface>
-      </collision>
-    </link>
-  </xacro:macro>
-  <xacro:turbo_link name="base_link" mesh_file="base_link.STL"
-    mass="0.0505669" ixx="1.585e-05" ixy="-6.321e-12" ixz="3.060e-11" iyy="3.953e-05" iyz="-3.073e-06" izz="3.988e-05"
-    size="0.1 0.05 0.05" xyz="0 0 -0.01" rpy="0 0 0" />
-  <xacro:turbo_link name="base_hip_middle_link" mesh_file="base_hip_middle_link.STL"
-    mass="0.3190303" ixx="0.0004755" ixy="-2.146e-07" ixz="-2.408e-08" iyy="0.0008352" iyz="4.645e-07" izz="0.0005132"
-    size="0.08 0.05 0.15" xyz="0 0 0.08" rpy="0 0 0" />
-  <xacro:turbo_link name="hip_head_link" mesh_file="hip_head_link.STL"
-    mass="0.1143471" ixx="2.400e-05" ixy="1.049e-10" ixz="-9.674e-09" iyy="2.959e-05" iyz="8.148e-08" izz="2.516e-05"
-    size="0.08 0.08 0.08" xyz="0 0 0" rpy="0 0 0" />
-  <xacro:turbo_link name="base_hip_left_link" mesh_file="base_hip_left_link.STL"
-    mass="0.107894" ixx="1.748e-05" ixy="-5.426e-11" ixz="-3.522e-22" iyy="2.777e-05" iyz="-1.556e-10" izz="1.748e-05"
-    size="0.04 0.04 0.04" xyz="0 0 0" rpy="0 0 0" />
-  <xacro:turbo_link name="hip_hip_left_link" mesh_file="hip_hip_left_link.STL"
-    mass="0.024442" ixx="1.327e-05" ixy="3.643e-07" ixz="4.214e-14" iyy="5.279e-06" iyz="-2.609e-10" izz="1.136e-05"
-    size="0.03 0.06 0.03" xyz="0 -0.03 0" rpy="0 0 0" />
-  <xacro:turbo_link name="hip_knee_left_link" mesh_file="hip_knee_left_link.STL"
-    mass="0.130204" ixx="4.591e-05" ixy="-2.099e-10" ixz="-4.142e-20" iyy="2.028e-05" iyz="-3.819e-21" izz="3.285e-05"
-    size="0.04 0.12 0.04" xyz="0 -0.05 0" rpy="0 0 0" />
-  <xacro:turbo_link name="knee_ankle_left_link" mesh_file="knee_ankle_left_link.STL"
-    mass="0.029851" ixx="9.566e-06" ixy="1.647e-06" ixz="4.489e-07" iyy="1.004e-05" iyz="-1.447e-06" izz="9.639e-06"
-    size="0.03 0.10 0.03" xyz="0 -0.05 0" rpy="0 0 0" />
-  <link name="ankle_ankle_left_link">
-    <inertial>
-      <origin xyz="-0.008 -0.007 -0.021" rpy="0 0 0" />
-      <mass value="0.085005" />
-      <inertia ixx="2.805e-05" ixy="5.987e-07" ixz="-9.674e-09" iyy="4.730e-05" iyz="5.071e-11" izz="2.353e-05" />
-    </inertial>
-    <visual>
-      <origin xyz="0 0 0" rpy="0 0 0" />
-      <geometry> <mesh filename="package://ros2_pkg/urdf/meshes/ankle_ankle_left_link.STL" /> </geometry>
-      <material name=""><color rgba="0.9 0.7 0.1 1" /></material>
-    </visual>
-    <collision>
-      <origin xyz="0 -0.02 -0.023" rpy="0 0 0" />
-      <geometry>
-        <box size="0.05 0.08 0.015" />
-      </geometry>
-      <surface>
-        <friction>
-          <ode>
-            <mu>${silicone_mu}</mu>
-            <mu2>${silicone_mu}</mu2>
-            <kp>${silicone_kp}</kp>
-            <kd>${silicone_kd}</kd>
-          </ode>
-        </friction>
-      </surface>
-    </collision>
-  </link>
-  <xacro:turbo_link name="base_hip_right_link" mesh_file="base_hip_right_link.STL"
-    mass="0.107894" ixx="1.748e-05" ixy="5.426e-11" ixz="-5.975e-21" iyy="2.777e-05" iyz="-1.556e-10" izz="1.748e-05"
-    size="0.04 0.04 0.04" xyz="0 0 0" rpy="0 0 0" />
-  <xacro:turbo_link name="hip_hip_right_link" mesh_file="hip_hip_right_link.STL"
-    mass="0.024442" ixx="1.327e-05" ixy="-3.643e-07" ixz="-4.023e-14" iyy="5.279e-06" iyz="2.609e-10" izz="1.136e-05"
-    size="0.03 0.06 0.03" xyz="0 -0.03 0" rpy="0 0 0" />
-  <xacro:turbo_link name="hip_knee_right_link" mesh_file="hip_knee_right_link.STL"
-    mass="0.130204" ixx="4.591e-05" ixy="-2.099e-10" ixz="-4.243e-20" iyy="2.028e-05" iyz="-5.559e-21" izz="3.285e-05"
-    size="0.04 0.12 0.04" xyz="0 -0.05 0" rpy="0 0 0" />
-  <xacro:turbo_link name="knee_ankle_right_link" mesh_file="knee_ankle_right_link.STL"
-    mass="0.029851" ixx="9.566e-06" ixy="1.647e-06" ixz="4.489e-07" iyy="1.004e-05" iyz="-1.447e-06" izz="9.639e-06"
-    size="0.03 0.10 0.03" xyz="0 -0.05 0" rpy="0 0 0" />
-  <link name="ankle_ankle_right_link">
-    <inertial>
-      <origin xyz="-0.008 -0.007 -0.022" rpy="0 0 0" />
-      <mass value="0.085921" />
-      <inertia ixx="2.807e-05" ixy="5.987e-07" ixz="-9.674e-09" iyy="4.732e-05" iyz="5.071e-11" izz="2.358e-05" />
-    </inertial>
-    <visual>
-      <origin xyz="0 0 0" rpy="0 0 0" />
-      <geometry> <mesh filename="package://ros2_pkg/urdf/meshes/ankle_ankle_right_link.STL" /> </geometry>
-      <material name=""><color rgba="0.9 0.7 0.1 1" /></material>
-    </visual>
-    <collision>
-      <origin xyz="0 -0.02 -0.023" rpy="0 0 0" />
-      <geometry> <box size="0.05 0.08 0.015" /> </geometry>
-      <surface>
-        <friction>
-          <ode>
-            <mu>${silicone_mu}</mu>
-            <mu2>${silicone_mu}</mu2>
-            <kp>${silicone_kp}</kp>
-            <kd>${silicone_kd}</kd>
-          </ode>
-        </friction>
-      </surface>
-    </collision>
-  </link>
-  <xacro:turbo_link name="hip_shoulder_left_link" mesh_file="hip_shoulder_left_link.STL"
-    mass="0.054051" ixx="8.314e-06" ixy="-1.049e-10" ixz="9.674e-09" iyy="1.388e-05" iyz="5.071e-11" izz="9.169e-06"
-    size="0.04 0.04 0.04" xyz="0 0 0" rpy="0 0 0" />
-  <xacro:turbo_link name="shoulder_shoulder_left_link" mesh_file="shoulder_shoulder_left_link.STL"
-    mass="0.079490" ixx="2.283e-05" ixy="1.051e-10" ixz="9.674e-09" iyy="1.930e-05" iyz="2.102e-10" izz="2.192e-05"
-    size="0.04 0.04 0.04" xyz="0 0 0" rpy="0 0 0" />
-  <xacro:turbo_link name="shoulder_elbow_left_link" mesh_file="shoulder_elbow_left_link.STL"
-    mass="0.092212" ixx="2.301e-05" ixy="-1.355e-07" ixz="2.522e-07" iyy="1.153e-05" iyz="-8.002e-08" izz="1.897e-05"
-    size="0.03 0.10 0.03" xyz="0 -0.04 0" rpy="0 0 0" />
-  <xacro:turbo_link name="hip_shoulder_right_link" mesh_file="hip_shoulder_right_link.STL"
-    mass="0.054051" ixx="8.314e-06" ixy="1.049e-10" ixz="-9.674e-09" iyy="1.388e-05" iyz="5.071e-11" izz="9.169e-06"
-    size="0.04 0.04 0.04" xyz="0 0 0" rpy="0 0 0" />
-  <xacro:turbo_link name="shoulder_shoulder_right_link" mesh_file="shoulder_shoulder_right_link.STL"
-    mass="0.079490" ixx="2.283e-05" ixy="1.051e-10" ixz="-9.674e-09" iyy="1.930e-05" iyz="3.116e-10" izz="2.192e-05"
-    size="0.04 0.04 0.04" xyz="0 0 0" rpy="0 0 0" />
-  <xacro:turbo_link name="shoulder_elbow_right_link" mesh_file="shoulder_elbow_right_link.STL"
-    mass="0.092163" ixx="2.298e-05" ixy="-9.310e-08" ixz="-2.271e-07" iyy="1.153e-05" iyz="-8.058e-08" izz="1.894e-05"
-    size="0.03 0.10 0.03" xyz="0 -0.04 0" rpy="0 0 0" />
-  <joint name="base_hip_left_joint" type="revolute">
-    <origin xyz="-0.035 -0.0205 -0.027" rpy="1.5708 0 -3.1416" />
-    <parent link="base_link" />
-    <child link="base_hip_left_link" />
-    <axis xyz="0 0 1" />
-    <limit lower="-0.17453" upper="0.69813" effort="1.08" velocity="6.16" />
-  </joint>
-  <joint name="hip_hip_left_joint" type="revolute">
-    <origin xyz="0.0295 -0.0205 0.0105" rpy="0 1.5708 0" />
-    <parent link="base_hip_left_link" />
-    <child link="hip_hip_left_link" />
-    <axis xyz="0 0 -1" />
-    <limit lower="-0.8" upper="0.69813" effort="1.08" velocity="6.16" />
-  </joint>
-  <joint name="hip_knee_left_joint" type="revolute">
-    <origin xyz="0 -0.06 0" rpy="0 0 0" />
-    <parent link="hip_hip_left_link" />
-    <child link="hip_knee_left_link" />
-    <axis xyz="0 0 -1" />
-    <limit lower="-1.3963" upper="1.3963" effort="1.08" velocity="6.16" />
-  </joint>
-  <joint name="knee_ankle_left_joint" type="revolute">
-    <origin xyz="0 -0.1034 0" rpy="0 0 0" />
-    <parent link="hip_knee_left_link" />
-    <child link="knee_ankle_left_link" />
-    <axis xyz="0 0 -1" />
-    <limit lower="-0.8" upper="0.8" effort="1.08" velocity="6.16" />
-  </joint>
-  <joint name="ankle_ankle_left_joint" type="revolute">
-    <origin xyz="0.0215 -0.057 -0.018" rpy="0 1.5708 0" />
-    <parent link="knee_ankle_left_link" />
-    <child link="ankle_ankle_left_link" />
-    <axis xyz="0 0 -1" />
-    <limit lower="-1.2217" upper="1.2217" effort="1.08" velocity="6.16" />
-  </joint>
-  <joint name="base_hip_right_joint" type="revolute">
-    <origin xyz="0.035 -0.0205 -0.027" rpy="1.5708 0 0" />
-    <parent link="base_link" />
-    <child link="base_hip_right_link" />
-    <axis xyz="0 0 -1" />
-    <limit lower="-0.69813" upper="0.17453" effort="1.08" velocity="6.16" />
-  </joint>
-  <joint name="hip_hip_right_joint" type="revolute">
-    <origin xyz="0.0309 -0.0205 -0.0126" rpy="0 1.5708 0" />
-    <parent link="base_hip_right_link" />
-    <child link="hip_hip_right_link" />
-    <axis xyz="0 0 -1" />
-    <limit lower="-0.69813" upper="0.8" effort="1.08" velocity="6.16" />
-  </joint>
-  <joint name="hip_knee_right_joint" type="revolute">
-    <origin xyz="0 -0.06 0" rpy="0 0 0" />
-    <parent link="hip_hip_right_link" />
-    <child link="hip_knee_right_link" />
-    <axis xyz="0 0 -1" />
-    <limit lower="-1.3963" upper="1.3963" effort="1.08" velocity="6.16" />
-  </joint>
-  <joint name="knee_ankle_right_joint" type="revolute">
-    <origin xyz="0 -0.1034 0" rpy="0 0 0" />
-    <parent link="hip_knee_right_link" />
-    <child link="knee_ankle_right_link" />
-    <axis xyz="0 0 -1" />
-    <limit lower="-0.8" upper="0.8" effort="1.08" velocity="6.16" />
-  </joint>
-  <joint name="ankle_ankle_right_joint" type="revolute">
-    <origin xyz="0.0215 -0.057 -0.0215" rpy="0 1.5708 0" />
-    <parent link="knee_ankle_right_link" />
-    <child link="ankle_ankle_right_link" />
-    <axis xyz="0 0 -1" />
-    <limit lower="-1.2217" upper="1.2217" effort="1.08" velocity="6.16" />
-  </joint>
-  <joint name="base_hip_middle_joint" type="revolute">
-    <origin xyz="0 0 0.0048" rpy="0 0 0" />
-    <parent link="base_link" />
-    <child link="base_hip_middle_link" />
-    <axis xyz="0 0 1" />
-    <limit lower="-0.5236" upper="0.5236" effort="1.08" velocity="6.16" />
-  </joint>
-  <joint name="hip_head_joint" type="fixed">
-    <origin xyz="0.001 -0.0017 0.1446" rpy="0 0 0" />
-    <parent link="base_hip_middle_link" />
-    <child link="hip_head_link" />
-  </joint>
-  <joint name="hip_shoulder_left_joint" type="revolute">
-    <origin xyz="-0.108 0.0195 0.1093" rpy="1.5708 0 0" />
-    <parent link="base_hip_middle_link" /> <child link="hip_shoulder_left_link" />
-    <axis xyz="0 0 1" /> <limit lower="-1.2" upper="0.2" effort="1" velocity="6"/>
-  </joint>
-  <joint name="shoulder_shoulder_left_joint" type="revolute">
-    <origin xyz="-0.015 -0.016 0.03" rpy="0 1.5708 0" />
-    <parent link="hip_shoulder_left_link" /> <child link="shoulder_shoulder_left_link" />
-    <axis xyz="0 0 -1" /> <limit lower="-1" upper="1" effort="1" velocity="6"/>
-  </joint>
-  <joint name="shoulder_elbow_left_joint" type="revolute">
-    <origin xyz="0 -0.063 0.026" rpy="0 0 0" />
-    <parent link="shoulder_shoulder_left_link" /> <child link="shoulder_elbow_left_link" />
-    <axis xyz="0 0 -1" /> <limit lower="-1.3" upper="1.3" effort="1" velocity="6"/>
-  </joint>
-  <joint name="hip_shoulder_right_joint" type="revolute">
-    <origin xyz="0.108 0.016 0.1093" rpy="1.5708 0 3.1416" />
-    <parent link="base_hip_middle_link" /> <child link="hip_shoulder_right_link" />
-    <axis xyz="0 0 -1" /> <limit lower="-0.2" upper="1.2" effort="1" velocity="6"/>
-  </joint>
-  <joint name="shoulder_shoulder_right_joint" type="revolute">
-    <origin xyz="-0.015 -0.016 -0.027" rpy="0 1.5708 0" />
-    <parent link="hip_shoulder_right_link" /> <child link="shoulder_shoulder_right_link" />
-    <axis xyz="0 0 -1" /> <limit lower="-1" upper="1" effort="1" velocity="6"/>
-  </joint>
-  <joint name="shoulder_elbow_right_joint" type="revolute">
-    <origin xyz="0 -0.063 0.026" rpy="0 0 0" />
-    <parent link="shoulder_shoulder_right_link" /> <child link="shoulder_elbow_right_link" />
-    <axis xyz="0 0 -1" /> <limit lower="-1.3" upper="1.3" effort="1" velocity="6"/>
-  </joint>
-  <gazebo reference="base_hip_middle_link">
-    <sensor name="imu_sensor" type="imu">
-      <always_on>1</always_on>
-      <update_rate>100</update_rate>
-      <visualize>true</visualize>
-      <topic>imu</topic>
-    </sensor>
-  </gazebo>
-  <xacro:robot_brain />
-</robot>
+/home/du/Desktop/NCKH_2026/Software/Ros2_WS/src/ros2_pkg/urdf/main_turbo.xacro
