Commit message: changed to 70D input PPO

File: Software/Ros2_WS/src/ros2_pkg/urdf/humanoid_physics.xacro (robot description, xacro)
@@ -44,13 +44,13 @@
     </gazebo>
     <xacro:setup_joint joint_name="base_hip_left_joint"/>
-    <xacro:make_controller joint_name="base_hip_left_joint"    p="8000" d="40"/>
+    <xacro:make_controller joint_name="base_hip_left_joint"    p="2000" d="20"/>
     <xacro:setup_joint joint_name="hip_hip_left_joint"/>
-    <xacro:make_controller joint_name="hip_hip_left_joint"     p="8000" d="40"/>
+    <xacro:make_controller joint_name="hip_hip_left_joint"     p="2000" d="20"/>
     <xacro:setup_joint joint_name="hip_knee_left_joint"/>
-    <xacro:make_controller joint_name="hip_knee_left_joint"    p="8000" d="40"/>
+    <xacro:make_controller joint_name="hip_knee_left_joint"    p="2000" d="20"/>
     <xacro:setup_joint joint_name="knee_ankle_left_joint"/>
-    <xacro:make_controller joint_name="knee_ankle_left_joint"  p="8000" d="40"/>
+    <xacro:make_controller joint_name="knee_ankle_left_joint"  p="2000" d="20"/>
     <xacro:setup_joint joint_name="ankle_ankle_left_joint"/>
-    <xacro:make_controller joint_name="ankle_ankle_left_joint" p="8000" d="40"/>
+    <xacro:make_controller joint_name="ankle_ankle_left_joint" p="2000" d="20"/>
     <gazebo reference="ankle_ankle_left_link">
       <mu1>${silicone_mu}</mu1>
@@ -61,13 +61,13 @@
     </gazebo>
     <xacro:setup_joint joint_name="base_hip_right_joint"/>
-    <xacro:make_controller joint_name="base_hip_right_joint"    p="8000" d="40"/>
+    <xacro:make_controller joint_name="base_hip_right_joint"    p="2000" d="20"/>
     <xacro:setup_joint joint_name="hip_hip_right_joint"/>
-    <xacro:make_controller joint_name="hip_hip_right_joint"     p="8000" d="40"/>
+    <xacro:make_controller joint_name="hip_hip_right_joint"     p="2000" d="20"/>
     <xacro:setup_joint joint_name="hip_knee_right_joint"/>
-    <xacro:make_controller joint_name="hip_knee_right_joint"    p="8000" d="40"/>
+    <xacro:make_controller joint_name="hip_knee_right_joint"    p="2000" d="20"/>
     <xacro:setup_joint joint_name="knee_ankle_right_joint"/>
-    <xacro:make_controller joint_name="knee_ankle_right_joint"  p="8000" d="40"/>
+    <xacro:make_controller joint_name="knee_ankle_right_joint"  p="2000" d="20"/>
     <xacro:setup_joint joint_name="ankle_ankle_right_joint"/>
-    <xacro:make_controller joint_name="ankle_ankle_right_joint" p="8000" d="40"/>
+    <xacro:make_controller joint_name="ankle_ankle_right_joint" p="2000" d="20"/>
     <gazebo reference="ankle_ankle_right_link">
       <mu1>${silicone_mu}</mu1>
@@ -78,17 +78,17 @@
     </gazebo>
     <xacro:setup_joint joint_name="base_hip_middle_joint"/>
-    <xacro:make_controller joint_name="base_hip_middle_joint"   p="8000" d="40"/>
+    <xacro:make_controller joint_name="base_hip_middle_joint"   p="2000" d="20"/>
     <xacro:setup_joint joint_name="hip_shoulder_left_joint"/>
-    <xacro:make_controller joint_name="hip_shoulder_left_joint"      p="8000" d="40"/>
+    <xacro:make_controller joint_name="hip_shoulder_left_joint"      p="2000" d="20"/>
     <xacro:setup_joint joint_name="shoulder_shoulder_left_joint"/>
-    <xacro:make_controller joint_name="shoulder_shoulder_left_joint" p="8000" d="40"/>
+    <xacro:make_controller joint_name="shoulder_shoulder_left_joint" p="2000" d="20"/>
     <xacro:setup_joint joint_name="shoulder_elbow_left_joint"/>
-    <xacro:make_controller joint_name="shoulder_elbow_left_joint"    p="8000" d="40"/>
+    <xacro:make_controller joint_name="shoulder_elbow_left_joint"    p="2000" d="20"/>
     <xacro:setup_joint joint_name="hip_shoulder_right_joint"/>
-    <xacro:make_controller joint_name="hip_shoulder_right_joint"      p="8000" d="40"/>
+    <xacro:make_controller joint_name="hip_shoulder_right_joint"      p="2000" d="20"/>
     <xacro:setup_joint joint_name="shoulder_shoulder_right_joint"/>
-    <xacro:make_controller joint_name="shoulder_shoulder_right_joint" p="8000" d="40"/>
+    <xacro:make_controller joint_name="shoulder_shoulder_right_joint" p="2000" d="20"/>
     <xacro:setup_joint joint_name="shoulder_elbow_right_joint"/>
-    <xacro:make_controller joint_name="shoulder_elbow_right_joint"    p="8000" d="40"/>
+    <xacro:make_controller joint_name="shoulder_elbow_right_joint"    p="2000" d="20"/>
   </xacro:macro>
 </robot>

Commit message: fix v2

File: Software/Ros2_WS/install/ros2_pkg/share/ros2_pkg/urdf/humanoid_physics.xacro (robot description, xacro)
@@ -1 +1,90 @@
-/home/du/Desktop/NCKH_2026/Software/Ros2_WS/src/ros2_pkg/urdf/humanoid_physics.xacro
+<?xml version="1.0"?>
+<robot xmlns:xacro="http://www.ros.org/wiki/xacro">
+  <xacro:property name="petg_mu" value="0.9" />
+  <xacro:property name="petg_kp" value="100000.0" />
+  <xacro:property name="petg_kd" value="10.0" />
+  <xacro:macro name="setup_joint" params="joint_name">
+    <gazebo reference="${joint_name}">
+      <implicitSpringDamper>true</implicitSpringDamper>
+    </gazebo>
+  </xacro:macro>
+  <xacro:macro name="setup_link" params="link_name">
+    <gazebo reference="${link_name}">
+      <mu1>${petg_mu}</mu1>
+      <mu2>${petg_mu}</mu2>
+      <kp>${petg_kp}</kp>
+      <kd>${petg_kd}</kd>
+      <self_collide>false</self_collide>
+    </gazebo>
+  </xacro:macro>
+<xacro:macro name="make_controller" params="joint_name p d">
+    <gazebo>
+      <plugin filename="gz-sim-joint-position-controller-system"
+              name="gz::sim::systems::JointPositionController">
+        <joint_name>${joint_name}</joint_name>
+        <topic>/model/humanoid_robot/joint/${joint_name}/cmd_pos</topic>
+        <p_gain>${p}</p_gain>
+        <i_gain>0.0</i_gain> <d_gain>${d}</d_gain>
+        <cmd_max>2.5</cmd_max>
+        <cmd_min>-2.5</cmd_min>
+        <velocity_max>2.5</velocity_max>
+      </plugin>
+    </gazebo>
+  </xacro:macro>
+  <xacro:macro name="robot_brain">
+    <gazebo>
+      <plugin filename="gz-sim-joint-state-publisher-system" name="gz::sim::systems::JointStatePublisher">
+        <update_rate>100</update_rate>
+      </plugin>
+      <plugin filename="gz-sim-imu-system" name="gz::sim::systems::Imu"></plugin>
+    </gazebo>
+    <xacro:setup_joint joint_name="base_hip_left_joint"/>
+    <xacro:make_controller joint_name="base_hip_left_joint"    p="2000" d="20"/>
+    <xacro:setup_joint joint_name="hip_hip_left_joint"/>
+    <xacro:make_controller joint_name="hip_hip_left_joint"     p="2000" d="20"/>
+    <xacro:setup_joint joint_name="hip_knee_left_joint"/>
+    <xacro:make_controller joint_name="hip_knee_left_joint"    p="2000" d="20"/>
+    <xacro:setup_joint joint_name="knee_ankle_left_joint"/>
+    <xacro:make_controller joint_name="knee_ankle_left_joint"  p="2000" d="20"/>
+    <xacro:setup_joint joint_name="ankle_ankle_left_joint"/>
+    <xacro:make_controller joint_name="ankle_ankle_left_joint" p="2000" d="20"/>
+    <gazebo reference="ankle_ankle_left_link">
+      <mu1>3.0</mu1>
+      <mu2>3.0</mu2>
+      <kp>100000</kp>
+      <kd>10</kd>
+      <self_collide>false</self_collide>
+    </gazebo>
+    <xacro:setup_joint joint_name="base_hip_right_joint"/>
+    <xacro:make_controller joint_name="base_hip_right_joint"    p="2000" d="20"/>
+    <xacro:setup_joint joint_name="hip_hip_right_joint"/>
+    <xacro:make_controller joint_name="hip_hip_right_joint"     p="2000" d="20"/>
+    <xacro:setup_joint joint_name="hip_knee_right_joint"/>
+    <xacro:make_controller joint_name="hip_knee_right_joint"    p="2000" d="20"/>
+    <xacro:setup_joint joint_name="knee_ankle_right_joint"/>
+    <xacro:make_controller joint_name="knee_ankle_right_joint"  p="2000" d="20"/>
+    <xacro:setup_joint joint_name="ankle_ankle_right_joint"/>
+    <xacro:make_controller joint_name="ankle_ankle_right_joint" p="2000" d="20"/>
+    <gazebo reference="ankle_ankle_right_link">
+      <mu1>3.0</mu1>
+      <mu2>3.0</mu2>
+      <kp>100000</kp>
+      <kd>10</kd>
+      <self_collide>false</self_collide>
+    </gazebo>
+    <xacro:setup_joint joint_name="base_hip_middle_joint"/>
+    <xacro:make_controller joint_name="base_hip_middle_joint"   p="2000" d="20"/>
+    <xacro:setup_joint joint_name="hip_shoulder_left_joint"/>
+    <xacro:make_controller joint_name="hip_shoulder_left_joint"      p="2000" d="20"/>
+    <xacro:setup_joint joint_name="shoulder_shoulder_left_joint"/>
+    <xacro:make_controller joint_name="shoulder_shoulder_left_joint" p="2000" d="20"/>
+    <xacro:setup_joint joint_name="shoulder_elbow_left_joint"/>
+    <xacro:make_controller joint_name="shoulder_elbow_left_joint"    p="2000" d="20"/>
+    <xacro:setup_joint joint_name="hip_shoulder_right_joint"/>
+    <xacro:make_controller joint_name="hip_shoulder_right_joint"      p="2000" d="20"/>
+    <xacro:setup_joint joint_name="shoulder_shoulder_right_joint"/>
+    <xacro:make_controller joint_name="shoulder_shoulder_right_joint" p="2000" d="20"/>
+    <xacro:setup_joint joint_name="shoulder_elbow_right_joint"/>
+    <xacro:make_controller joint_name="shoulder_elbow_right_joint"    p="2000" d="20"/>
+  </xacro:macro>
+</robot>

File: Software/Ros2_WS/install/ros2_pkg/share/ros2_pkg/urdf/main.xacro (robot description, xacro)
@@ -1 +1,39 @@
-/home/du/Desktop/NCKH_2026/Software/Ros2_WS/src/ros2_pkg/urdf/main.xacro
+<?xml version="1.0"?>
+<robot name="robot_humanoid" xmlns:xacro="http://www.ros.org/wiki/xacro">
+  <xacro:include filename="$(find ros2_pkg)/urdf/urdf/Robot.urdf" />
+  <xacro:include filename="$(find ros2_pkg)/urdf/humanoid_physics.xacro" />
+  <link name="base_footprint"/>
+  <joint name="base_footprint_joint" type="fixed">
+    <parent link="base_footprint"/>
+    <child link="base_link"/>
+    <origin xyz="0 0 0" rpy="0 0 0"/>
+  </joint>
+  <xacro:setup_link link_name="base_link" />
+  <xacro:setup_link link_name="base_hip_middle_link" />
+  <xacro:setup_link link_name="hip_head_link" />
+  <xacro:setup_link link_name="base_hip_left_link" />
+  <xacro:setup_link link_name="hip_hip_left_link" />
+  <xacro:setup_link link_name="hip_knee_left_link" />
+  <xacro:setup_link link_name="knee_ankle_left_link" />
+  <!-- ankle_ankle_left_link: friction đặt riêng trong humanoid_physics.xacro -->
+  <xacro:setup_link link_name="base_hip_right_link" />
+  <xacro:setup_link link_name="hip_hip_right_link" />
+  <xacro:setup_link link_name="hip_knee_right_link" />
+  <xacro:setup_link link_name="knee_ankle_right_link" />
+  <!-- ankle_ankle_right_link: friction đặt riêng trong humanoid_physics.xacro -->
+  <xacro:setup_link link_name="hip_shoulder_left_link" />
+  <xacro:setup_link link_name="shoulder_shoulder_left_link" />
+  <xacro:setup_link link_name="shoulder_elbow_left_link" />
+  <xacro:setup_link link_name="hip_shoulder_right_link" />
+  <xacro:setup_link link_name="shoulder_shoulder_right_link" />
+  <xacro:setup_link link_name="shoulder_elbow_right_link" />
+  <gazebo reference="base_hip_middle_link">
+    <sensor name="imu_sensor" type="imu">
+      <always_on>1</always_on> <update_rate>100</update_rate>
+      <visualize>true</visualize>
+      <topic>imu</topic>
+      <pose>0 0 0 0 0 0</pose>
+    </sensor>
+  </gazebo>
+  <xacro:robot_brain />
+</robot>

File: Software/Ros2_WS/src/ros2_pkg/urdf/humanoid_physics.xacro (robot description, xacro)
@@ -4,8 +4,4 @@
   <xacro:property name="petg_kp" value="100000.0" />
   <xacro:property name="petg_kd" value="10.0" />
-  <xacro:property name="silicone_mu" value="0.99" />
-  <xacro:property name="silicone_kp" value="100000.0" />
-  <xacro:property name="silicone_kd" value="10.0" />
-  <xacro:property name="silicone_thickness" value="0.002" />
   <xacro:macro name="setup_joint" params="joint_name">
     <gazebo reference="${joint_name}">
@@ -32,5 +28,5 @@
         <cmd_max>2.5</cmd_max>
         <cmd_min>-2.5</cmd_min>
-        <velocity_max>6.0</velocity_max>
+        <velocity_max>2.5</velocity_max>
       </plugin>
     </gazebo>
@@ -54,8 +50,8 @@
     <xacro:make_controller joint_name="ankle_ankle_left_joint" p="2000" d="20"/>
     <gazebo reference="ankle_ankle_left_link">
-      <mu1>${silicone_mu}</mu1>
-      <mu2>${silicone_mu}</mu2>
-      <kp>${silicone_kp}</kp>
-      <kd>${silicone_kd}</kd>
+      <mu1>3.0</mu1>
+      <mu2>3.0</mu2>
+      <kp>100000</kp>
+      <kd>10</kd>
       <self_collide>false</self_collide>
     </gazebo>
@@ -71,8 +67,8 @@
     <xacro:make_controller joint_name="ankle_ankle_right_joint" p="2000" d="20"/>
     <gazebo reference="ankle_ankle_right_link">
-      <mu1>${silicone_mu}</mu1>
-      <mu2>${silicone_mu}</mu2>
-      <kp>${silicone_kp}</kp>
-      <kd>${silicone_kd}</kd>
+      <mu1>3.0</mu1>
+      <mu2>3.0</mu2>
+      <kp>100000</kp>
+      <kd>10</kd>
       <self_collide>false</self_collide>
     </gazebo>

File: Software/Ros2_WS/src/ros2_pkg/urdf/main.xacro (robot description, xacro)
@@ -16,10 +16,10 @@
   <xacro:setup_link link_name="hip_knee_left_link" />
   <xacro:setup_link link_name="knee_ankle_left_link" />
-  <xacro:setup_link link_name="ankle_ankle_left_link" />
+  <!-- ankle_ankle_left_link: friction đặt riêng trong humanoid_physics.xacro -->
   <xacro:setup_link link_name="base_hip_right_link" />
   <xacro:setup_link link_name="hip_hip_right_link" />
   <xacro:setup_link link_name="hip_knee_right_link" />
   <xacro:setup_link link_name="knee_ankle_right_link" />
-  <xacro:setup_link link_name="ankle_ankle_right_link" />
+  <!-- ankle_ankle_right_link: friction đặt riêng trong humanoid_physics.xacro -->
   <xacro:setup_link link_name="hip_shoulder_left_link" />
   <xacro:setup_link link_name="shoulder_shoulder_left_link" />

File: Software/Ros2_WS_v2/install/ros2_pkg_v2/share/ros2_pkg_v2/urdf/main.xacro (robot description, xacro)
@@ -133,5 +133,5 @@
   <gazebo>
     <plugin filename="gz_ros2_control-system" name="gz_ros2_control::GazeboSimROS2ControlPlugin">
-      <parameters>$(find ros2_pkg_v2)/config/controller_config.yaml</parameters>
+      <parameters>$(find ros2_pkg_v2)/config/controller_config_v2.yaml</parameters>
       <hold_joints>true</hold_joints>
     </plugin>
