Commit message: add uvc test

File: Software/Ros2_WS/install/ros2_pkg/share/ros2_pkg/urdf/urdf/Robot.urdf (robot description, URDF)
Before this commit: robot Robot, 19 links, 18 joints
Links:
- link hip_hip_left_link: mass 0.0782857304964655 -> 0.0782857304964654
- link hip_hip_right_link: mass 0.0782857304964655 -> 0.0782857304964656
- link hip_knee_left_link: mass 0.0763616529215024 -> 0.130204487078614
- link hip_knee_right_link: mass 0.0763616529215023 -> 0.130204487078614
- link hip_shoulder_left_link: mass 0.054051364576062 -> 0.0540513645760621
- link shoulder_elbow_left_link: mass 0.0947347359064563 -> 0.0922123668839718
- link shoulder_elbow_right_link: mass 0.09468264272445 -> 0.0921635034792499
Joints:
- joint ankle_ankle_right_joint: origin xyz=0.0214999999999963 -0.0570000000000002 -0.0215000000000039 rpy=0 1.5707963267949 0 -> xyz=0.0215 -0.057 -0.0215 rpy=0 1.5708 0
- joint base_hip_right_joint: origin xyz=0.0350000000000045 -0.0204999999999993 -0.027 rpy=1.5707963267949 0 0 -> xyz=0.035 -0.0205 -0.027 rpy=1.5708 0 0
- joint hip_knee_left_joint: origin xyz=0 -0.0599999999999997 0 rpy=0 0 0 -> xyz=0 -0.06 0 rpy=0 0 0
- joint hip_knee_right_joint: origin xyz=0 -0.0600000000000001 0 rpy=0 0 0 -> xyz=0 -0.06 0 rpy=0 0 0
- joint knee_knee_left_joint: origin xyz=0.0215 -0.0570000000000001 -0.0180000000000003 rpy=0 1.5707963267949 0 -> xyz=0.0215 -0.057 -0.018 rpy=0 1.5708 0

Commit message: fix uvc

File: Software/Ros2_WS/install/ros2_pkg/share/ros2_pkg/urdf/urdf/Robot.urdf (robot description, URDF)
Before this commit: robot Robot, 19 links, 18 joints
Links:
- removed link knee_knee_left_link
- added link ankle_ankle_left_link, mass 0.0850053645760622; collision mesh filename=package://ros2_pkg/urdf/meshes/ankle_ankle_left_link.STL; visual mesh filename=package://ros2_pkg/urdf/meshes/ankle_ankle_left_link.STL
- link hip_shoulder_left_link: mass 0.0540513645760621 -> 0.054051364576062
Joints:
- removed joint knee_knee_left_joint
- added joint ankle_ankle_left_joint: type revolute, parent knee_ankle_left_link, child ankle_ankle_left_link, origin xyz=0.0215 -0.0570000000000001 -0.0180000000000003 rpy=0 1.5707963267949 0, axis 0 0 -1, limit lower=-1.2217 upper=1.2217 effort=0.8 velocity=6.16
- joint ankle_ankle_right_joint: limit lower=-1.2217 upper=1.2217 effort=2.5 velocity=6.16 -> lower=-1.2217 upper=1.2217 effort=0.8 velocity=6.16; origin xyz=0.0215 -0.057 -0.0215 rpy=0 1.5708 0 -> xyz=0.0214999999999963 -0.0570000000000002 -0.0215000000000039 rpy=0 1.5707963267949 0
- joint base_hip_left_joint: limit lower=-0.17453 upper=0.69813 effort=2.5 velocity=6.16 -> lower=-0.17453 upper=0.69813 effort=0.8 velocity=6.16
- joint base_hip_middle_joint: limit lower=-0.5236 upper=0.5236 effort=2.5 velocity=6.16 -> lower=-0.5236 upper=0.5236 effort=0.8 velocity=6.16; origin xyz=0 0 0.00479999999999899 rpy=0 0 0 -> xyz=0 0 0.0048 rpy=0 0 0
- joint base_hip_right_joint: limit lower=-0.69813 upper=0.17453 effort=2.5 velocity=6.16 -> lower=-0.69813 upper=0.17453 effort=0.8 velocity=6.16; origin xyz=0.035 -0.0205 -0.027 rpy=1.5708 0 0 -> xyz=0.0350000000000045 -0.0204999999999993 -0.027 rpy=1.5707963267949 0 0
- joint hip_hip_left_joint: limit lower=-0.5236 upper=0.69813 effort=2.5 velocity=6.16 -> lower=-0.5236 upper=0.69813 effort=0.8 velocity=6.16
- joint hip_hip_right_joint: limit lower=-0.69813 upper=0.5236 effort=2.5 velocity=6.16 -> lower=-0.69813 upper=0.5236 effort=0.8 velocity=6.16
- joint hip_knee_left_joint: limit lower=-1.3963 upper=1.3963 effort=2.5 velocity=6.16 -> lower=-1.3963 upper=1.3963 effort=0.8 velocity=6.16; origin xyz=0 -0.06 0 rpy=0 0 0 -> xyz=0 -0.0599999999999997 0 rpy=0 0 0
- joint hip_knee_right_joint: limit lower=-1.3963 upper=1.3963 effort=2.5 velocity=6.16 -> lower=-1.3963 upper=1.3963 effort=0.8 velocity=6.16; origin xyz=0 -0.06 0 rpy=0 0 0 -> xyz=0 -0.0600000000000001 0 rpy=0 0 0
- joint hip_shoulder_left_joint: limit lower=-1.2217 upper=0.17453 effort=2.5 velocity=6.16 -> lower=-1.2217 upper=0.17453 effort=0.8 velocity=6.16
- joint hip_shoulder_right_joint: limit lower=-0.17453 upper=1.2217 effort=2.5 velocity=6.16 -> lower=-0.17453 upper=1.2217 effort=0.8 velocity=6.16; origin xyz=0.108 0.0159999999999952 0.1093 rpy=1.5707963267949 0 3.14159265358979 -> xyz=0.108 0.016 0.1093 rpy=1.5708 0 3.1416
- joint knee_ankle_left_joint: limit lower=-0.34907 upper=0.69813 effort=2.5 velocity=6.16 -> lower=-0.34907 upper=0.69813 effort=0.8 velocity=6.16
- joint knee_ankle_right_joint: limit lower=-0.69813 upper=0.34907 effort=2.5 velocity=6.16 -> lower=-0.69813 upper=0.34907 effort=0.8 velocity=6.16
- joint shoulder_elbow_left_joint: limit lower=-1.3963 upper=1.3963 effort=2.5 velocity=6.16 -> lower=-1.3963 upper=1.3963 effort=0.8 velocity=6.16; origin xyz=0 -0.0636218145435769 0.0261724872211921 rpy=0 0 0 -> xyz=0 -0.063622 0.026172 rpy=0 0 0
- joint shoulder_elbow_right_joint: limit lower=-1.3963 upper=1.3963 effort=2.5 velocity=6.16 -> lower=-1.3963 upper=1.3963 effort=0.8 velocity=6.16; origin xyz=0 -0.0636218145435714 0.0261724872211919 rpy=0 0 0 -> xyz=0 -0.063622 0.026172 rpy=0 0 0
- joint shoulder_shoulder_left_joint: limit lower=-1.0472 upper=1.0472 effort=2.5 velocity=6.16 -> lower=-1.0472 upper=1.0472 effort=0.8 velocity=6.16
- joint shoulder_shoulder_right_joint: limit lower=-1.0472 upper=1.0472 effort=2.5 velocity=6.16 -> lower=-1.0472 upper=1.0472 effort=0.8 velocity=6.16; origin xyz=-0.0156724872211916 -0.0168781854564282 -0.0273999999999952 rpy=0 1.5707963267949 0 -> xyz=-0.015672 -0.016878 -0.0274 rpy=0 1.5708 0

File: Software/Ros2_WS/src/ros2_pkg/urdf/humanoid_physics.xacro (robot description, xacro)
@@ -2,5 +2,6 @@
 <robot xmlns:xacro="http://www.ros.org/wiki/xacro">
   <xacro:property name="petg_mu" value="0.7" />
-  <xacro:property name="petg_kp" value="100000.0" /> <xacro:property name="petg_kd" value="1.0" />
+  <xacro:property name="petg_kp" value="100000.0" />
+  <xacro:property name="petg_kd" value="1.0" />
   <xacro:macro name="setup_link" params="link_name">
     <gazebo reference="${link_name}">
@@ -9,5 +10,29 @@
       <kp>${petg_kp}</kp>
       <kd>${petg_kd}</kd>
-      <auto_inertia_params><mass>0.15</mass></auto_inertia_params>
+    </gazebo>
+  </xacro:macro>
+  <xacro:macro name="setup_joint" params="joint_name">
+    <gazebo reference="${joint_name}">
+      <implicitSpringDamper>true</implicitSpringDamper>
+      <springStiffness>15.0</springStiffness>
+      <springReference>0.0</springReference>
+      <friction>1.5</friction>
+      <damping>1.0</damping>
+    </gazebo>
+  </xacro:macro>
+  <xacro:macro name="make_controller" params="joint_name p d">
+    <gazebo>
+      <plugin filename="gz-sim-joint-position-controller-system"
+              name="gz::sim::systems::JointPositionController">
+        <joint_name>${joint_name}</joint_name>
+        <topic>/model/humanoid_robot/joint/${joint_name}/cmd_pos</topic>
+        <p_gain>${p}</p_gain>
+        <i_gain>0.1</i_gain>
+        <d_gain>${d}</d_gain>
+        <i_max>10</i_max>
+        <i_min>-10</i_min>
+        <cmd_max>200.0</cmd_max>
+        <cmd_min>-200.0</cmd_min>
+      </plugin>
     </gazebo>
   </xacro:macro>
@@ -15,29 +40,42 @@
     <gazebo>
       <plugin filename="gz-sim-joint-state-publisher-system" name="gz::sim::systems::JointStatePublisher">
-        <update_rate>100</update_rate>
+        <update_rate>500</update_rate>
       </plugin>
-      <plugin filename="gz-sim-joint-trajectory-controller-system" name="gz::sim::systems::JointTrajectoryController">
-        <topic>/model/humanoid_robot/joint_trajectory</topic>
-        <gains joint_name="hip_knee_left_joint">    <p>5000</p> <d>50</d> <i_clamp>0</i_clamp> <max_force>6.0</max_force> </gains>
-        <gains joint_name="hip_knee_right_joint">   <p>5000</p> <d>50</d> <i_clamp>0</i_clamp> <max_force>6.0</max_force> </gains>
-        <gains joint_name="knee_ankle_left_joint">  <p>5000</p> <d>50</d> <i_clamp>0</i_clamp> <max_force>6.0</max_force> </gains>
-        <gains joint_name="knee_ankle_right_joint"> <p>5000</p> <d>50</d> <i_clamp>0</i_clamp> <max_force>6.0</max_force> </gains>
-        <gains joint_name="hip_hip_left_joint">     <p>5000</p> <d>50</d> <i_clamp>0</i_clamp> <max_force>6.0</max_force> </gains>
-        <gains joint_name="hip_hip_right_joint">    <p>5000</p> <d>50</d> <i_clamp>0</i_clamp> <max_force>6.0</max_force> </gains>
-        <gains joint_name="base_hip_left_joint">    <p>5000</p> <d>50</d> </gains>
-        <gains joint_name="base_hip_right_joint">   <p>5000</p> <d>50</d> </gains>
-        <gains joint_name="base_hip_middle_joint">  <p>5000</p> <d>50</d> </gains>
-        <gains joint_name="knee_knee_left_joint">   <p>5000</p> <d>50</d> </gains>
-        <gains joint_name="ankle_ankle_right_joint"><p>5000</p> <d>50</d> </gains>
-        </plugin>
       <plugin filename="gz-sim-imu-system" name="gz::sim::systems::Imu"></plugin>
     </gazebo>
-  </xacro:macro>
-  <xacro:macro name="setup_joint" params="joint_name">
-    <gazebo reference="${joint_name}">
-      <implicitSpringDamper>true</implicitSpringDamper>
-      <friction>0.1</friction>
-      <damping>0.1</damping>
-    </gazebo>
+    <xacro:setup_joint joint_name="base_hip_left_joint"/>
+    <xacro:setup_joint joint_name="hip_hip_left_joint"/>
+    <xacro:setup_joint joint_name="hip_knee_left_joint"/>
+    <xacro:setup_joint joint_name="knee_ankle_left_joint"/>
+    <xacro:setup_joint joint_name="ankle_ankle_left_joint"/>
+    <xacro:make_controller joint_name="base_hip_left_joint"    p="5000" d="100"/>
+    <xacro:make_controller joint_name="hip_hip_left_joint"     p="5000" d="100"/>
+    <xacro:make_controller joint_name="hip_knee_left_joint"    p="8000" d="200"/>
+    <xacro:make_controller joint_name="knee_ankle_left_joint"  p="8000" d="200"/>
+    <xacro:make_controller joint_name="ankle_ankle_left_joint" p="5000" d="100"/>
+    <xacro:setup_joint joint_name="base_hip_right_joint"/>
+    <xacro:setup_joint joint_name="hip_hip_right_joint"/>
+    <xacro:setup_joint joint_name="hip_knee_right_joint"/>
+    <xacro:setup_joint joint_name="knee_ankle_right_joint"/>
+    <xacro:setup_joint joint_name="ankle_ankle_right_joint"/>
+    <xacro:make_controller joint_name="base_hip_right_joint"    p="5000" d="100"/>
+    <xacro:make_controller joint_name="hip_hip_right_joint"     p="5000" d="100"/>
+    <xacro:make_controller joint_name="hip_knee_right_joint"    p="8000" d="200"/>
+    <xacro:make_controller joint_name="knee_ankle_right_joint"  p="8000" d="200"/>
+    <xacro:make_controller joint_name="ankle_ankle_right_joint" p="5000" d="100"/>
+    <xacro:setup_joint joint_name="base_hip_middle_joint"/>
+    <xacro:make_controller joint_name="base_hip_middle_joint"   p="5000" d="100"/>
+    <xacro:setup_joint joint_name="hip_shoulder_left_joint"/>
+    <xacro:setup_joint joint_name="shoulder_shoulder_left_joint"/>
+    <xacro:setup_joint joint_name="shoulder_elbow_left_joint"/>
+    <xacro:make_controller joint_name="hip_shoulder_left_joint"      p="1500" d="50"/>
+    <xacro:make_controller joint_name="shoulder_shoulder_left_joint" p="1500" d="50"/>
+    <xacro:make_controller joint_name="shoulder_elbow_left_joint"    p="1500" d="50"/>
+    <xacro:setup_joint joint_name="hip_shoulder_right_joint"/>
+    <xacro:setup_joint joint_name="shoulder_shoulder_right_joint"/>
+    <xacro:setup_joint joint_name="shoulder_elbow_right_joint"/>
+    <xacro:make_controller joint_name="hip_shoulder_right_joint"      p="1500" d="50"/>
+    <xacro:make_controller joint_name="shoulder_shoulder_right_joint" p="1500" d="50"/>
+    <xacro:make_controller joint_name="shoulder_elbow_right_joint"    p="1500" d="50"/>
   </xacro:macro>
 </robot>

File: Software/Ros2_WS/src/ros2_pkg/urdf/main.xacro (robot description, xacro)
@@ -1,10 +1,4 @@
 <?xml version="1.0"?>
 <robot name="robot_humanoid" xmlns:xacro="http://www.ros.org/wiki/xacro">
-  <link name="world_root"/>
-  <joint name="world_root_joint" type="fixed">
-    <parent link="world_root"/>
-    <child link="base_link"/>
-    <origin xyz="0 0 0" rpy="0 0 0"/>
-  </joint>
   <xacro:include filename="$(find ros2_pkg)/urdf/urdf/Robot.urdf" />
   <xacro:include filename="$(find ros2_pkg)/urdf/humanoid_physics.xacro" />
@@ -16,5 +10,5 @@
   <xacro:setup_link link_name="hip_knee_left_link" />
   <xacro:setup_link link_name="knee_ankle_left_link" />
-  <xacro:setup_link link_name="knee_knee_left_link" />
+  <xacro:setup_link link_name="ankle_ankle_left_link" />
   <xacro:setup_link link_name="base_hip_right_link" />
   <xacro:setup_link link_name="hip_hip_right_link" />
@@ -28,27 +22,13 @@
   <xacro:setup_link link_name="shoulder_shoulder_right_link" />
   <xacro:setup_link link_name="shoulder_elbow_right_link" />
-  <gazebo reference="hip_head_link">
+  <gazebo reference="base_hip_middle_link">
     <sensor name="imu_sensor" type="imu">
       <always_on>1</always_on>
-      <update_rate>100</update_rate>
+      <update_rate>500</update_rate>
       <visualize>true</visualize>
       <topic>imu</topic>
+      <pose>0 0 0 0 0 0</pose>
     </sensor>
   </gazebo>
   <xacro:robot_brain />
-  <xacro:setup_joint joint_name="base_hip_middle_joint" />
-  <xacro:setup_joint joint_name="base_hip_left_joint" />
-  <xacro:setup_joint joint_name="base_hip_right_joint" />
-  <xacro:setup_joint joint_name="hip_hip_left_joint" />
-  <xacro:setup_joint joint_name="hip_knee_left_joint" />
-  <xacro:setup_joint joint_name="knee_ankle_left_joint" />
-  <xacro:setup_joint joint_name="knee_knee_left_joint" /> <xacro:setup_joint joint_name="hip_hip_right_joint" />
-  <xacro:setup_joint joint_name="hip_knee_right_joint" />
-  <xacro:setup_joint joint_name="knee_ankle_right_joint" />
-  <xacro:setup_joint joint_name="ankle_ankle_right_joint" /> <xacro:setup_joint joint_name="hip_shoulder_left_joint" />
-  <xacro:setup_joint joint_name="shoulder_shoulder_left_joint" />
-  <xacro:setup_joint joint_name="shoulder_elbow_left_joint" />
-  <xacro:setup_joint joint_name="hip_shoulder_right_joint" />
-  <xacro:setup_joint joint_name="shoulder_shoulder_right_joint" />
-  <xacro:setup_joint joint_name="shoulder_elbow_right_joint" />
 </robot>

File: Software/Ros2_WS/src/ros2_pkg/urdf/urdf/Robot.urdf (robot description, URDF)
Before this commit: robot Robot, 19 links, 18 joints
Links:
- link ankle_ankle_left_link: geometry collision mesh filename=package://ros2_pkg/urdf/meshes/ankle_ankle_left_link.STL; visual mesh filename=package://ros2_pkg/urdf/meshes/ankle_ankle_left_link.STL
- link ankle_ankle_right_link: geometry collision mesh filename=package://ros2_pkg/urdf/meshes/ankle_ankle_right_link.STL; visual mesh filename=package://ros2_pkg/urdf/meshes/ankle_ankle_right_link.STL
- link base_hip_left_link: geometry collision mesh filename=package://ros2_pkg/urdf/meshes/base_hip_left_link.STL; visual mesh filename=package://ros2_pkg/urdf/meshes/base_hip_left_link.STL
- link base_hip_middle_link: geometry collision mesh filename=package://ros2_pkg/urdf/meshes/base_hip_middle_link.STL; visual mesh filename=package://ros2_pkg/urdf/meshes/base_hip_middle_link.STL
- link base_hip_right_link: geometry collision mesh filename=package://ros2_pkg/urdf/meshes/base_hip_right_link.STL; visual mesh filename=package://ros2_pkg/urdf/meshes/base_hip_right_link.STL
- link base_link: geometry collision mesh filename=package://ros2_pkg/urdf/meshes/base_link.STL; visual mesh filename=package://ros2_pkg/urdf/meshes/base_link.STL
- link hip_head_link: geometry collision mesh filename=package://ros2_pkg/urdf/meshes/hip_head_link.STL; visual mesh filename=package://ros2_pkg/urdf/meshes/hip_head_link.STL
- link hip_hip_left_link: geometry collision mesh filename=package://ros2_pkg/urdf/meshes/hip_hip_left_link.STL; visual mesh filename=package://ros2_pkg/urdf/meshes/hip_hip_left_link.STL
- link hip_hip_right_link: geometry collision mesh filename=package://ros2_pkg/urdf/meshes/hip_hip_right_link.STL; visual mesh filename=package://ros2_pkg/urdf/meshes/hip_hip_right_link.STL
- link hip_knee_left_link: geometry collision mesh filename=package://ros2_pkg/urdf/meshes/hip_knee_left_link.STL; visual mesh filename=package://ros2_pkg/urdf/meshes/hip_knee_left_link.STL
- link hip_knee_right_link: geometry collision mesh filename=package://ros2_pkg/urdf/meshes/hip_knee_right_link.STL; visual mesh filename=package://ros2_pkg/urdf/meshes/hip_knee_right_link.STL
- link hip_shoulder_left_link: geometry collision mesh filename=package://ros2_pkg/urdf/meshes/hip_shoulder_left_link.STL; visual mesh filename=package://ros2_pkg/urdf/meshes/hip_shoulder_left_link.STL
- link hip_shoulder_right_link: geometry collision mesh filename=package://ros2_pkg/urdf/meshes/hip_shoulder_right_link.STL; visual mesh filename=package://ros2_pkg/urdf/meshes/hip_shoulder_right_link.STL
- link knee_ankle_left_link: geometry collision mesh filename=package://ros2_pkg/urdf/meshes/knee_ankle_left_link.STL; visual mesh filename=package://ros2_pkg/urdf/meshes/knee_ankle_left_link.STL
- link knee_ankle_right_link: geometry collision mesh filename=package://ros2_pkg/urdf/meshes/knee_ankle_right_link.STL; visual mesh filename=package://ros2_pkg/urdf/meshes/knee_ankle_right_link.STL
- link shoulder_elbow_left_link: geometry collision mesh filename=package://ros2_pkg/urdf/meshes/shoulder_elbow_left_link.STL; visual mesh filename=package://ros2_pkg/urdf/meshes/shoulder_elbow_left_link.STL
- link shoulder_elbow_right_link: geometry collision mesh filename=package://ros2_pkg/urdf/meshes/shoulder_elbow_right_link.STL; visual mesh filename=package://ros2_pkg/urdf/meshes/shoulder_elbow_right_link.STL
- link shoulder_shoulder_left_link: geometry collision mesh filename=package://ros2_pkg/urdf/meshes/shoulder_shoulder_left_link.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; visual mesh filename=package://ros2_pkg/urdf/meshes/shoulder_shoulder_left_link.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
- link shoulder_shoulder_right_link: geometry collision mesh filename=package://ros2_pkg/urdf/meshes/shoulder_shoulder_right_link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; visual mesh filename=package://ros2_pkg/urdf/meshes/shoulder_shoulder_right_link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
Joints:
- joint ankle_ankle_left_joint: limit lower=-1.2217 upper=1.2217 effort=1.08 velocity=6.16 -> lower=-1.2217 upper=1.2217 effort=0.8 velocity=6.16
- joint ankle_ankle_right_joint: limit lower=-1.2217 upper=1.2217 effort=1.08 velocity=6.16 -> lower=-1.2217 upper=1.2217 effort=0.8 velocity=6.16
- joint base_hip_left_joint: limit lower=-0.17453 upper=0.69813 effort=1.08 velocity=6.16 -> lower=-0.17453 upper=0.69813 effort=0.8 velocity=6.16
- joint base_hip_middle_joint: limit lower=-0.5236 upper=0.5236 effort=1.08 velocity=6.16 -> lower=-0.5236 upper=0.5236 effort=0.8 velocity=6.16
- joint base_hip_right_joint: limit lower=-0.69813 upper=0.17453 effort=1.08 velocity=6.16 -> lower=-0.69813 upper=0.17453 effort=0.8 velocity=6.16
- joint hip_hip_left_joint: limit lower=-0.5236 upper=0.69813 effort=1.08 velocity=6.16 -> lower=-0.5236 upper=0.69813 effort=0.8 velocity=6.16
- joint hip_hip_right_joint: limit lower=-0.69813 upper=0.5236 effort=1.08 velocity=6.16 -> lower=-0.69813 upper=0.5236 effort=0.8 velocity=6.16
- joint hip_knee_left_joint: limit lower=-1.3963 upper=1.3963 effort=1.08 velocity=6.16 -> lower=-1.3963 upper=1.3963 effort=0.8 velocity=6.16
- joint hip_knee_right_joint: limit lower=-1.3963 upper=1.3963 effort=1.08 velocity=6.16 -> lower=-1.3963 upper=1.3963 effort=0.8 velocity=6.16
- joint hip_shoulder_left_joint: limit lower=-1.2217 upper=0.17453 effort=1.08 velocity=6.16 -> lower=-1.2217 upper=0.17453 effort=0.8 velocity=6.16
- joint hip_shoulder_right_joint: limit lower=-0.17453 upper=1.2217 effort=1.08 velocity=6.16 -> lower=-0.17453 upper=1.2217 effort=0.8 velocity=6.16
- joint knee_ankle_left_joint: limit lower=-0.34907 upper=0.69813 effort=1.08 velocity=6.16 -> lower=-0.34907 upper=0.69813 effort=0.8 velocity=6.16
- joint knee_ankle_right_joint: limit lower=-0.69813 upper=0.34907 effort=1.08 velocity=6.16 -> lower=-0.69813 upper=0.34907 effort=0.8 velocity=6.16
- joint shoulder_elbow_left_joint: limit lower=-1.3963 upper=1.3963 effort=1.08 velocity=6.16 -> lower=-1.3963 upper=1.3963 effort=0.8 velocity=6.16
- joint shoulder_elbow_right_joint: limit lower=-1.3963 upper=1.3963 effort=1.08 velocity=6.16 -> lower=-1.3963 upper=1.3963 effort=0.8 velocity=6.16
- joint shoulder_shoulder_left_joint: limit lower=-1.0472 upper=1.0472 effort=1.08 velocity=6.16 -> lower=-1.0472 upper=1.0472 effort=0.8 velocity=6.16
- joint shoulder_shoulder_right_joint: limit lower=-1.0472 upper=1.0472 effort=1.08 velocity=6.16 -> lower=-1.0472 upper=1.0472 effort=0.8 velocity=6.16
