Commit message: fix urdf(hand)

File: Software/Ros2_WS/src/ros2_pkg/urdf/urdf/Robot.urdf (robot description, URDF)
Before this commit: robot Robot, 19 links, 18 joints
Links:
- link base_hip_left_link: mass 0.0540513645760621 -> 0.054051
- link base_hip_middle_link: mass 0.322024415361419 -> 0
- link base_hip_right_link: mass 0.054051364576062 -> 0.054051
- link base_link: mass 0.0505669356625173 -> 0.050567
- link hip_hip_left_link: mass 0.0782857304964655 -> 0.078286
- link hip_hip_right_link: mass 0.0782857304964655 -> 0.0782857304964656
- link hip_knee_left_link: mass 0.0763616529215024 -> 0.076362
- link hip_shoulder_left_link: mass 0.054051364576062 -> 0.054051
- link hip_shoulder_right_link: mass 0.054051364576062 -> 0.054051
- link knee_ankle_left_link: mass 0.0298519989099933 -> 0.029852
- link knee_ankle_right_link: mass 0.0298519989099933 -> 0.0298519989099934
- link shoulder_elbow_left_link: mass 0.0947347359064563 -> 0.092212
- link shoulder_elbow_right_link: mass 0.09468264272445 -> 0.092164
- link shoulder_shoulder_left_link: mass 0.0794907034391992 -> 0.079491
- link shoulder_shoulder_right_link: mass 0.0794907034391992 -> 0.079491
Joints:
- joint base_hip_left_joint: origin xyz=-0.0350000000000001 -0.0204999999999994 -0.0270000000000001 rpy=1.57079632679489 0 -3.14159265358979 -> xyz=-0.035 -0.0205 -0.027 rpy=1.5708 0 -3.1416
- joint base_hip_right_joint: origin xyz=0.0350000000000045 -0.0204999999999993 -0.027 rpy=1.5707963267949 0 0 -> xyz=0.035 -0.0205 -0.027 rpy=1.5708 0 0

Commit message: fix urdf(servo)

File: Software/Ros2_WS/src/ros2_pkg/urdf/urdf/Robot.urdf (robot description, URDF)
Before this commit: robot Robot, 19 links, 18 joints
Links:
- link base_hip_left_link: mass 0.054051 -> 0.0540513645760621
- link base_hip_middle_link: mass 0 -> 0.322024415361419
- link base_hip_right_link: mass 0.054051 -> 0.054051364576062
- link base_link: mass 0.050567 -> 0.0505669356625173
- link hip_hip_left_link: mass 0.078286 -> 0.0782857304964654
- link hip_knee_left_link: mass 0.076362 -> 0.130204487078614
- link hip_knee_right_link: mass 0.0763616529215023 -> 0.130204487078614
- link hip_shoulder_left_link: mass 0.054051 -> 0.0540513645760621
- link hip_shoulder_right_link: mass 0.054051 -> 0.054051364576062
- link knee_ankle_left_link: mass 0.029852 -> 0.0298519989099933
- link knee_ankle_right_link: mass 0.0298519989099934 -> 0.0298519989099933
- link shoulder_elbow_left_link: mass 0.092212 -> 0.0922123668839718
- link shoulder_elbow_right_link: mass 0.092164 -> 0.0921635034792499
- link shoulder_shoulder_left_link: mass 0.079491 -> 0.0794907034391992
- link shoulder_shoulder_right_link: mass 0.079491 -> 0.0794907034391992
Joints:
- joint ankle_ankle_right_joint: origin xyz=0.0214999999999963 -0.0570000000000002 -0.0215000000000039 rpy=0 1.5707963267949 0 -> xyz=0.0215 -0.057 -0.0215 rpy=0 1.5708 0
- joint base_hip_left_joint: origin xyz=-0.035 -0.0205 -0.027 rpy=1.5708 0 -3.1416 -> xyz=-0.0350000000000001 -0.0204999999999994 -0.0270000000000001 rpy=1.57079632679489 0 -3.14159265358979
- joint hip_knee_left_joint: origin xyz=0 -0.0599999999999997 0 rpy=0 0 0 -> xyz=0 -0.06 0 rpy=0 0 0
- joint hip_knee_right_joint: origin xyz=0 -0.0600000000000001 0 rpy=0 0 0 -> xyz=0 -0.06 0 rpy=0 0 0
- joint knee_knee_left_joint: origin xyz=0.0215 -0.0570000000000001 -0.0180000000000003 rpy=0 1.5707963267949 0 -> xyz=0.0215 -0.057 -0.018 rpy=0 1.5708 0

Commit message: fix rviz.launch.py

File: Software/Ros2_WS/src/ros2_pkg/urdf/urdf/Robot.urdf (robot description, URDF)
Before this commit: robot Robot, 19 links, 18 joints
Links:
- link ankle_ankle_right_link: geometry collision mesh filename=package://ros2_pkg/urdf/meshes/ankle_ankle_right_link.STL; visual mesh filename=package://ros2_pkg/urdf/meshes/ankle_ankle_right_link.STL
- link base_hip_left_link: geometry collision mesh filename=package://ros2_pkg/urdf/meshes/base_hip_left_link.STL; visual mesh filename=package://ros2_pkg/urdf/meshes/base_hip_left_link.STL
- link base_hip_middle_link: geometry collision mesh filename=package://ros2_pkg/urdf/meshes/base_hip_middle_link.STL; visual mesh filename=package://ros2_pkg/urdf/meshes/base_hip_middle_link.STL
- link base_hip_right_link: geometry collision mesh filename=package://ros2_pkg/urdf/meshes/base_hip_right_link.STL; visual mesh filename=package://ros2_pkg/urdf/meshes/base_hip_right_link.STL
- link base_link: geometry collision mesh filename=package://ros2_pkg/urdf/meshes/base_link.STL; visual mesh filename=package://ros2_pkg/urdf/meshes/base_link.STL
- link hip_head_link: geometry collision mesh filename=package://ros2_pkg/urdf/meshes/hip_head_link.STL; visual mesh filename=package://ros2_pkg/urdf/meshes/hip_head_link.STL
- link hip_hip_left_link: geometry collision mesh filename=package://ros2_pkg/urdf/meshes/hip_hip_left_link.STL; visual mesh filename=package://ros2_pkg/urdf/meshes/hip_hip_left_link.STL
- link hip_hip_right_link: geometry collision mesh filename=package://ros2_pkg/urdf/meshes/hip_hip_right_link.STL; visual mesh filename=package://ros2_pkg/urdf/meshes/hip_hip_right_link.STL
- link hip_knee_left_link: geometry collision mesh filename=package://ros2_pkg/urdf/meshes/hip_knee_left_link.STL; visual mesh filename=package://ros2_pkg/urdf/meshes/hip_knee_left_link.STL
- link hip_knee_right_link: geometry collision mesh filename=package://ros2_pkg/urdf/meshes/hip_knee_right_link.STL; visual mesh filename=package://ros2_pkg/urdf/meshes/hip_knee_right_link.STL
- link hip_shoulder_left_link: geometry collision mesh filename=package://ros2_pkg/urdf/meshes/hip_shoulder_left_link.STL; visual mesh filename=package://ros2_pkg/urdf/meshes/hip_shoulder_left_link.STL
- link hip_shoulder_right_link: geometry collision mesh filename=package://ros2_pkg/urdf/meshes/hip_shoulder_right_link.STL; visual mesh filename=package://ros2_pkg/urdf/meshes/hip_shoulder_right_link.STL
- link knee_ankle_left_link: geometry collision mesh filename=package://ros2_pkg/urdf/meshes/knee_ankle_left_link.STL; visual mesh filename=package://ros2_pkg/urdf/meshes/knee_ankle_left_link.STL
- link knee_ankle_right_link: geometry collision mesh filename=package://ros2_pkg/urdf/meshes/knee_ankle_right_link.STL; visual mesh filename=package://ros2_pkg/urdf/meshes/knee_ankle_right_link.STL
- link knee_knee_left_link: geometry collision mesh filename=package://ros2_pkg/urdf/meshes/knee_knee_left_link.STL; visual mesh filename=package://ros2_pkg/urdf/meshes/knee_knee_left_link.STL
- link shoulder_elbow_left_link: geometry collision mesh filename=package://ros2_pkg/urdf/meshes/shoulder_elbow_left_link.STL; visual mesh filename=package://ros2_pkg/urdf/meshes/shoulder_elbow_left_link.STL
- link shoulder_elbow_right_link: geometry collision mesh filename=package://ros2_pkg/urdf/meshes/shoulder_elbow_right_link.STL; visual mesh filename=package://ros2_pkg/urdf/meshes/shoulder_elbow_right_link.STL
- link shoulder_shoulder_left_link: geometry collision mesh filename=package://ros2_pkg/urdf/meshes/shoulder_shoulder_left_link.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; visual mesh filename=package://ros2_pkg/urdf/meshes/shoulder_shoulder_left_link.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
- link shoulder_shoulder_right_link: geometry collision mesh filename=package://ros2_pkg/urdf/meshes/shoulder_shoulder_right_link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; visual mesh filename=package://ros2_pkg/urdf/meshes/shoulder_shoulder_right_link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

Commit message: fix joint name

File: Software/Ros2_WS/src/ros2_pkg/urdf/urdf/Robot.urdf (robot description, URDF)
Before this commit: robot Robot, 19 links, 18 joints
Links:
- removed link knee_knee_left_link
- added link ankle_ankle_left_link, mass 0.0850053645760622; collision mesh filename=package://Robot/meshes/ankle_ankle_left_link.STL; visual mesh filename=package://Robot/meshes/ankle_ankle_left_link.STL
- link ankle_ankle_right_link: geometry collision mesh filename=package://Robot/meshes/ankle_ankle_right_link.STL; visual mesh filename=package://Robot/meshes/ankle_ankle_right_link.STL
- link base_hip_left_link: geometry collision mesh filename=package://Robot/meshes/base_hip_left_link.STL; visual mesh filename=package://Robot/meshes/base_hip_left_link.STL
- link base_hip_middle_link: geometry collision mesh filename=package://Robot/meshes/base_hip_middle_link.STL; visual mesh filename=package://Robot/meshes/base_hip_middle_link.STL
- link base_hip_right_link: geometry collision mesh filename=package://Robot/meshes/base_hip_right_link.STL; visual mesh filename=package://Robot/meshes/base_hip_right_link.STL
- link base_link: geometry collision mesh filename=package://Robot/meshes/base_link.STL; visual mesh filename=package://Robot/meshes/base_link.STL
- link hip_head_link: geometry collision mesh filename=package://Robot/meshes/hip_head_link.STL; visual mesh filename=package://Robot/meshes/hip_head_link.STL
- link hip_hip_left_link: geometry collision mesh filename=package://Robot/meshes/hip_hip_left_link.STL; visual mesh filename=package://Robot/meshes/hip_hip_left_link.STL
- link hip_hip_right_link: geometry collision mesh filename=package://Robot/meshes/hip_hip_right_link.STL; visual mesh filename=package://Robot/meshes/hip_hip_right_link.STL
- link hip_knee_left_link: geometry collision mesh filename=package://Robot/meshes/hip_knee_left_link.STL; visual mesh filename=package://Robot/meshes/hip_knee_left_link.STL
- link hip_knee_right_link: geometry collision mesh filename=package://Robot/meshes/hip_knee_right_link.STL; visual mesh filename=package://Robot/meshes/hip_knee_right_link.STL
- link hip_shoulder_left_link: mass 0.0540513645760621 -> 0.054051364576062; geometry collision mesh filename=package://Robot/meshes/hip_shoulder_left_link.STL; visual mesh filename=package://Robot/meshes/hip_shoulder_left_link.STL
- link hip_shoulder_right_link: geometry collision mesh filename=package://Robot/meshes/hip_shoulder_right_link.STL; visual mesh filename=package://Robot/meshes/hip_shoulder_right_link.STL
- link knee_ankle_left_link: geometry collision mesh filename=package://Robot/meshes/knee_ankle_left_link.STL; visual mesh filename=package://Robot/meshes/knee_ankle_left_link.STL
- link knee_ankle_right_link: geometry collision mesh filename=package://Robot/meshes/knee_ankle_right_link.STL; visual mesh filename=package://Robot/meshes/knee_ankle_right_link.STL
- link shoulder_elbow_left_link: geometry collision mesh filename=package://Robot/meshes/shoulder_elbow_left_link.STL; visual mesh filename=package://Robot/meshes/shoulder_elbow_left_link.STL
- link shoulder_elbow_right_link: geometry collision mesh filename=package://Robot/meshes/shoulder_elbow_right_link.STL; visual mesh filename=package://Robot/meshes/shoulder_elbow_right_link.STL
- link shoulder_shoulder_left_link: geometry collision mesh filename=package://Robot/meshes/shoulder_shoulder_left_link.STL; visual mesh filename=package://Robot/meshes/shoulder_shoulder_left_link.STL
- link shoulder_shoulder_right_link: geometry collision mesh filename=package://Robot/meshes/shoulder_shoulder_right_link.STL; visual mesh filename=package://Robot/meshes/shoulder_shoulder_right_link.STL
Joints:
- removed joint knee_knee_left_joint
- added joint ankle_ankle_left_joint: type revolute, parent knee_ankle_left_link, child ankle_ankle_left_link, origin xyz=0.0215 -0.0570000000000001 -0.0180000000000003 rpy=0 1.5707963267949 0, axis 0 0 -1, limit lower=-1.2217 upper=1.2217 effort=1.08 velocity=6.16
- joint ankle_ankle_right_joint: limit lower=-1.2217 upper=1.2217 effort=2.5 velocity=6.16 -> lower=-1.2217 upper=1.2217 effort=1.08 velocity=6.16; origin xyz=0.0215 -0.057 -0.0215 rpy=0 1.5708 0 -> xyz=0.0214999999999963 -0.0570000000000002 -0.0215000000000039 rpy=0 1.5707963267949 0
- joint base_hip_left_joint: limit lower=-0.17453 upper=0.69813 effort=2.5 velocity=6.16 -> lower=-0.17453 upper=0.69813 effort=1.08 velocity=6.16
- joint base_hip_middle_joint: limit lower=-0.5236 upper=0.5236 effort=2.5 velocity=6.16 -> lower=-0.5236 upper=0.5236 effort=1.08 velocity=6.16; origin xyz=0 0 0.00479999999999899 rpy=0 0 0 -> xyz=0 0 0.0048 rpy=0 0 0
- joint base_hip_right_joint: limit lower=-0.69813 upper=0.17453 effort=2.5 velocity=6.16 -> lower=-0.69813 upper=0.17453 effort=1.08 velocity=6.16; origin xyz=0.035 -0.0205 -0.027 rpy=1.5708 0 0 -> xyz=0.0350000000000045 -0.0204999999999993 -0.027 rpy=1.5707963267949 0 0
- joint hip_hip_left_joint: limit lower=-0.5236 upper=0.69813 effort=2.5 velocity=6.16 -> lower=-0.5236 upper=0.69813 effort=1.08 velocity=6.16
- joint hip_hip_right_joint: limit lower=-0.69813 upper=0.5236 effort=2.5 velocity=6.16 -> lower=-0.69813 upper=0.5236 effort=1.08 velocity=6.16
- joint hip_knee_left_joint: limit lower=-1.3963 upper=1.3963 effort=2.5 velocity=6.16 -> lower=-1.3963 upper=1.3963 effort=1.08 velocity=6.16; origin xyz=0 -0.06 0 rpy=0 0 0 -> xyz=0 -0.0599999999999997 0 rpy=0 0 0
- joint hip_knee_right_joint: limit lower=-1.3963 upper=1.3963 effort=2.5 velocity=6.16 -> lower=-1.3963 upper=1.3963 effort=1.08 velocity=6.16; origin xyz=0 -0.06 0 rpy=0 0 0 -> xyz=0 -0.0600000000000001 0 rpy=0 0 0
- joint hip_shoulder_left_joint: limit lower=-1.2217 upper=0.17453 effort=2.5 velocity=6.16 -> lower=-1.2217 upper=0.17453 effort=1.08 velocity=6.16
- joint hip_shoulder_right_joint: limit lower=-0.17453 upper=1.2217 effort=2.5 velocity=6.16 -> lower=-0.17453 upper=1.2217 effort=1.08 velocity=6.16; origin xyz=0.108 0.0159999999999952 0.1093 rpy=1.5707963267949 0 3.14159265358979 -> xyz=0.108 0.016 0.1093 rpy=1.5708 0 3.1416
- joint knee_ankle_left_joint: limit lower=-0.34907 upper=0.69813 effort=2.5 velocity=6.16 -> lower=-0.34907 upper=0.69813 effort=1.08 velocity=6.16
- joint knee_ankle_right_joint: limit lower=-0.69813 upper=0.34907 effort=2.5 velocity=6.16 -> lower=-0.69813 upper=0.34907 effort=1.08 velocity=6.16
- joint shoulder_elbow_left_joint: limit lower=-1.3963 upper=1.3963 effort=2.5 velocity=6.16 -> lower=-1.3963 upper=1.3963 effort=1.08 velocity=6.16; origin xyz=0 -0.0636218145435769 0.0261724872211921 rpy=0 0 0 -> xyz=0 -0.063622 0.026172 rpy=0 0 0
- joint shoulder_elbow_right_joint: limit lower=-1.3963 upper=1.3963 effort=2.5 velocity=6.16 -> lower=-1.3963 upper=1.3963 effort=1.08 velocity=6.16; origin xyz=0 -0.0636218145435714 0.0261724872211919 rpy=0 0 0 -> xyz=0 -0.063622 0.026172 rpy=0 0 0
- joint shoulder_shoulder_left_joint: limit lower=-1.0472 upper=1.0472 effort=2.5 velocity=6.16 -> lower=-1.0472 upper=1.0472 effort=1.08 velocity=6.16
- joint shoulder_shoulder_right_joint: limit lower=-1.0472 upper=1.0472 effort=2.5 velocity=6.16 -> lower=-1.0472 upper=1.0472 effort=1.08 velocity=6.16; origin xyz=-0.0156724872211916 -0.0168781854564282 -0.0273999999999952 rpy=0 1.5707963267949 0 -> xyz=-0.015672 -0.016878 -0.0274 rpy=0 1.5708 0

Commit message: fix urdf

File: Software/Ros2_WS/src/ros2_pkg/urdf/urdf/Robot.urdf (robot description, URDF)
Before this commit: robot Robot, 19 links, 18 joints
Links:
- link ankle_ankle_right_link: mass 0.0859210745449871 -> 0.085921074544987
- link base_hip_left_link: mass 0.0540513645760621 -> 0.107894198733174
- link base_hip_middle_link: mass 0.322024415361419 -> 0.319030319361419
- link base_hip_right_link: mass 0.054051364576062 -> 0.107894198733174
- link hip_hip_left_link: mass 0.0782857304964654 -> 0.0244428963393535
- link hip_hip_right_link: mass 0.0782857304964656 -> 0.0244428963393535
- link shoulder_shoulder_left_link: mass 0.0794907034391992 -> 0.0794907034391991
Joints:
- joint ankle_ankle_left_joint: limit lower=-1.2217 upper=1.2217 effort=0.8 velocity=6.16 -> lower=-1.2217 upper=1.2217 effort=1.08 velocity=6.16; origin xyz=0.0215 -0.0570000000000001 -0.0180000000000003 rpy=0 1.5707963267949 0 -> xyz=0.0215 -0.057 -0.018 rpy=0 1.5708 0
- joint ankle_ankle_right_joint: axis 0 0 -1 -> 0 0 1; limit lower=-1.2217 upper=1.2217 effort=0.8 velocity=6.16 -> lower=-1.2217 upper=1.2217 effort=1.08 velocity=6.16; origin xyz=0.0214999999999963 -0.0570000000000002 -0.0215000000000039 rpy=0 1.5707963267949 0 -> xyz=0.0215 -0.057 -0.0215 rpy=3.1416 -1.5708 0
- joint base_hip_left_joint: limit lower=-0.17453 upper=0.69813 effort=0.8 velocity=6.16 -> lower=-0.17453 upper=0.69813 effort=1.08 velocity=6.16; origin xyz=-0.0350000000000001 -0.0204999999999994 -0.0270000000000001 rpy=1.57079632679489 0 -3.14159265358979 -> xyz=-0.035 -0.0205 -0.027 rpy=1.5708 0 -3.1416
- joint base_hip_middle_joint: limit lower=-0.5236 upper=0.5236 effort=0.8 velocity=6.16 -> lower=-0.5236 upper=0.5236 effort=1.08 velocity=6.16; origin xyz=0 0 0.0048 rpy=0 0 0 -> xyz=0 0 0.00479999999999899 rpy=0 0 0
- joint base_hip_right_joint: limit lower=-0.69813 upper=0.17453 effort=0.8 velocity=6.16 -> lower=-0.69813 upper=0.17453 effort=1.08 velocity=6.16; origin xyz=0.0350000000000045 -0.0204999999999993 -0.027 rpy=1.5707963267949 0 0 -> xyz=0.035 -0.0205 -0.027 rpy=1.5708 0 0
- joint hip_hip_left_joint: limit lower=-0.8 upper=0.69813 effort=0.8 velocity=6.16 -> lower=-0.8 upper=0.69813 effort=1.08 velocity=6.16; origin xyz=0.0295 -0.0205000000000001 0.0105 rpy=0 1.5707963267949 0 -> xyz=0.0295 -0.0205 0.0105 rpy=0 1.5708 0
- joint hip_hip_right_joint: limit lower=-0.69813 upper=0.8 effort=0.8 velocity=6.16 -> lower=-0.69813 upper=0.8 effort=1.08 velocity=6.16; origin xyz=0.0309000000000001 -0.0204999999999999 -0.0126 rpy=0 1.5707963267949 0 -> xyz=0.0309 -0.0205 -0.0126 rpy=0 1.5708 0
- joint hip_knee_left_joint: limit lower=-1.3963 upper=1.3963 effort=0.8 velocity=6.16 -> lower=-1.3963 upper=1.3963 effort=1.08 velocity=6.16; origin xyz=0 -0.0599999999999997 0 rpy=0 0 0 -> xyz=0 -0.06 0 rpy=0 0 0
- joint hip_knee_right_joint: limit lower=-1.3963 upper=1.3963 effort=0.8 velocity=6.16 -> lower=-1.3963 upper=1.3963 effort=1.08 velocity=6.16; origin xyz=0 -0.0600000000000001 0 rpy=0 0 0 -> xyz=0 -0.06 0 rpy=0 0 0
- joint hip_shoulder_left_joint: limit lower=-1.2217 upper=0.17453 effort=0.8 velocity=6.16 -> lower=-1.2217 upper=0.17453 effort=1.08 velocity=6.16
- joint hip_shoulder_right_joint: limit lower=-0.17453 upper=1.2217 effort=0.8 velocity=6.16 -> lower=-0.17453 upper=1.2217 effort=1.08 velocity=6.16; origin xyz=0.108 0.016 0.1093 rpy=1.5708 0 3.1416 -> xyz=0.108 0.0159999999999952 0.1093 rpy=1.5707963267949 0 3.14159265358979
- joint knee_ankle_left_joint: limit lower=-0.8 upper=0.8 effort=0.8 velocity=6.16 -> lower=-0.8 upper=0.8 effort=1.08 velocity=6.16
- joint knee_ankle_right_joint: limit lower=-0.8 upper=0.8 effort=0.8 velocity=6.16 -> lower=-0.8 upper=0.8 effort=1.08 velocity=6.16
- joint shoulder_elbow_left_joint: limit lower=-1.3963 upper=1.3963 effort=0.8 velocity=6.16 -> lower=-1.3963 upper=1.3963 effort=1.08 velocity=6.16; origin xyz=0 -0.063622 0.026172 rpy=0 0 0 -> xyz=0 -0.0636218145435769 0.0261724872211921 rpy=0 0 0
- joint shoulder_elbow_right_joint: limit lower=-1.3963 upper=1.3963 effort=0.8 velocity=6.16 -> lower=-1.3963 upper=1.3963 effort=1.08 velocity=6.16; origin xyz=0 -0.063622 0.026172 rpy=0 0 0 -> xyz=0 -0.0636218145435714 0.0261724872211919 rpy=0 0 0
- joint shoulder_shoulder_left_joint: limit lower=-1.0472 upper=1.0472 effort=0.8 velocity=6.16 -> lower=-1.0472 upper=1.0472 effort=1.08 velocity=6.16
- joint shoulder_shoulder_right_joint: limit lower=-1.0472 upper=1.0472 effort=0.8 velocity=6.16 -> lower=-1.0472 upper=1.0472 effort=1.08 velocity=6.16; origin xyz=-0.015672 -0.016878 -0.0274 rpy=0 1.5708 0 -> xyz=-0.0156724872211916 -0.0168781854564282 -0.0273999999999952 rpy=0 1.5707963267949 0
