Commit message: fix urdf

File: Software/Ros2_WS/src/ros2_pkg/urdf/urdf/Robot.urdf (robot description, URDF)
Before this commit: robot Robot.urdf, 19 links, 18 joints
Links:
- link ankle_ankle_left_link: geometry collision mesh filename=package://Robot/meshes/ankle_ankle_left_link.STL; visual mesh filename=package://Robot/meshes/ankle_ankle_left_link.STL
- link ankle_ankle_right_link: mass 0.085921074544987 -> 0.0859210745449871; geometry collision mesh filename=package://Robot/meshes/ankle_ankle_right_link.STL; visual mesh filename=package://Robot/meshes/ankle_ankle_right_link.STL
- link base_hip_left_link: geometry collision mesh filename=package://Robot/meshes/base_hip_left_link.STL; visual mesh filename=package://Robot/meshes/base_hip_left_link.STL
- link base_hip_middle_link: geometry collision mesh filename=package://Robot/meshes/base_hip_middle_link.STL; visual mesh filename=package://Robot/meshes/base_hip_middle_link.STL
- link base_hip_right_link: geometry collision mesh filename=package://Robot/meshes/base_hip_right_link.STL; visual mesh filename=package://Robot/meshes/base_hip_right_link.STL
- link base_link: geometry collision mesh filename=package://Robot/meshes/base_link.STL; visual mesh filename=package://Robot/meshes/base_link.STL
- link hip_head_link: geometry collision mesh filename=package://Robot/meshes/hip_head_link.STL; visual mesh filename=package://Robot/meshes/hip_head_link.STL
- link hip_hip_left_link: geometry collision mesh filename=package://Robot/meshes/hip_hip_left_link.STL; visual mesh filename=package://Robot/meshes/hip_hip_left_link.STL
- link hip_hip_right_link: mass 0.0244428963393535 -> 0.0244428963393534; geometry collision mesh filename=package://Robot/meshes/hip_hip_right_link.STL; visual mesh filename=package://Robot/meshes/hip_hip_right_link.STL
- link hip_knee_left_link: geometry collision mesh filename=package://Robot/meshes/hip_knee_left_link.STL; visual mesh filename=package://Robot/meshes/hip_knee_left_link.STL
- link hip_knee_right_link: geometry collision mesh filename=package://Robot/meshes/hip_knee_right_link.STL; visual mesh filename=package://Robot/meshes/hip_knee_right_link.STL
- link hip_shoulder_left_link: geometry collision mesh filename=package://Robot/meshes/hip_shoulder_left_link.STL; visual mesh filename=package://Robot/meshes/hip_shoulder_left_link.STL
- link hip_shoulder_right_link: geometry collision mesh filename=package://Robot/meshes/hip_shoulder_right_link.STL; visual mesh filename=package://Robot/meshes/hip_shoulder_right_link.STL
- link knee_ankle_left_link: geometry collision mesh filename=package://Robot/meshes/knee_ankle_left_link.STL; visual mesh filename=package://Robot/meshes/knee_ankle_left_link.STL
- link knee_ankle_right_link: geometry collision mesh filename=package://Robot/meshes/knee_ankle_right_link.STL; visual mesh filename=package://Robot/meshes/knee_ankle_right_link.STL
- link shoulder_elbow_left_link: geometry collision mesh filename=package://Robot/meshes/shoulder_elbow_left_link.STL; visual mesh filename=package://Robot/meshes/shoulder_elbow_left_link.STL
- link shoulder_elbow_right_link: geometry collision mesh filename=package://Robot/meshes/shoulder_elbow_right_link.STL; visual mesh filename=package://Robot/meshes/shoulder_elbow_right_link.STL
- link shoulder_shoulder_left_link: mass 0.0794907034391991 -> 0.0794907034391992; geometry collision mesh filename=package://Robot/meshes/shoulder_shoulder_left_link.STL; visual mesh filename=package://Robot/meshes/shoulder_shoulder_left_link.STL
- link shoulder_shoulder_right_link: geometry collision mesh filename=package://Robot/meshes/shoulder_shoulder_right_link.STL; visual mesh filename=package://Robot/meshes/shoulder_shoulder_right_link.STL
Joints:
- joint ankle_ankle_left_joint: origin xyz=0.0215 -0.057 -0.018 rpy=0 1.5708 0 -> xyz=0.0215 -0.0570000000000001 -0.0180000000000003 rpy=0 1.5707963267949 0
- joint ankle_ankle_right_joint: axis 0 0 1 -> 0 0 -1; origin xyz=0.0215 -0.057 -0.0215 rpy=3.1416 -1.5708 0 -> xyz=0.0214999999999963 -0.0569999999999992 -0.0215000000000082 rpy=0 1.5707963267949 0
- joint base_hip_left_joint: origin xyz=-0.035 -0.0205 -0.027 rpy=1.5708 0 -3.1416 -> xyz=-0.0350000000000001 -0.0204999999999994 -0.0270000000000001 rpy=1.57079632679489 0 -3.14159265358979
- joint hip_hip_left_joint: origin xyz=0.0295 -0.0205 0.0105 rpy=0 1.5708 0 -> xyz=0.0295 -0.0205000000000001 0.0105 rpy=0 1.5707963267949 0
- joint hip_hip_right_joint: origin xyz=0.0309 -0.0205 -0.0126 rpy=0 1.5708 0 -> xyz=0.0309000000000001 -0.0204999999999999 -0.0126 rpy=0 1.5707963267949 0
- joint hip_knee_right_joint: origin xyz=0 -0.06 0 rpy=0 0 0 -> xyz=0 -0.0600000000000001 0 rpy=0 0 0

Commit message: o

File: Software/Ros2_WS/src/ros2_pkg/urdf/urdf/Robot.urdf (robot description, URDF)
Before this commit: robot Robot, 19 links, 18 joints
Links:
- link ankle_ankle_left_link: geometry collision mesh filename=package://ros2_pkg/urdf/meshes/ankle_ankle_left_link.STL; visual mesh filename=package://ros2_pkg/urdf/meshes/ankle_ankle_left_link.STL
- link ankle_ankle_right_link: geometry collision mesh filename=package://ros2_pkg/urdf/meshes/ankle_ankle_right_link.STL; visual mesh filename=package://ros2_pkg/urdf/meshes/ankle_ankle_right_link.STL
- link base_hip_left_link: geometry collision mesh filename=package://ros2_pkg/urdf/meshes/base_hip_left_link.STL; visual mesh filename=package://ros2_pkg/urdf/meshes/base_hip_left_link.STL
- link base_hip_middle_link: geometry collision mesh filename=package://ros2_pkg/urdf/meshes/base_hip_middle_link.STL; visual mesh filename=package://ros2_pkg/urdf/meshes/base_hip_middle_link.STL
- link base_hip_right_link: geometry collision mesh filename=package://ros2_pkg/urdf/meshes/base_hip_right_link.STL; visual mesh filename=package://ros2_pkg/urdf/meshes/base_hip_right_link.STL
- link base_link: geometry collision mesh filename=package://ros2_pkg/urdf/meshes/base_link.STL; visual mesh filename=package://ros2_pkg/urdf/meshes/base_link.STL
- link hip_head_link: geometry collision mesh filename=package://ros2_pkg/urdf/meshes/hip_head_link.STL; visual mesh filename=package://ros2_pkg/urdf/meshes/hip_head_link.STL
- link hip_hip_left_link: geometry collision mesh filename=package://ros2_pkg/urdf/meshes/hip_hip_left_link.STL; visual mesh filename=package://ros2_pkg/urdf/meshes/hip_hip_left_link.STL
- link hip_hip_right_link: geometry collision mesh filename=package://ros2_pkg/urdf/meshes/hip_hip_right_link.STL; visual mesh filename=package://ros2_pkg/urdf/meshes/hip_hip_right_link.STL
- link hip_knee_left_link: geometry collision mesh filename=package://ros2_pkg/urdf/meshes/hip_knee_left_link.STL; visual mesh filename=package://ros2_pkg/urdf/meshes/hip_knee_left_link.STL
- link hip_knee_right_link: geometry collision mesh filename=package://ros2_pkg/urdf/meshes/hip_knee_right_link.STL; visual mesh filename=package://ros2_pkg/urdf/meshes/hip_knee_right_link.STL
- link hip_shoulder_left_link: geometry collision mesh filename=package://ros2_pkg/urdf/meshes/hip_shoulder_left_link.STL; visual mesh filename=package://ros2_pkg/urdf/meshes/hip_shoulder_left_link.STL
- link hip_shoulder_right_link: geometry collision mesh filename=package://ros2_pkg/urdf/meshes/hip_shoulder_right_link.STL; visual mesh filename=package://ros2_pkg/urdf/meshes/hip_shoulder_right_link.STL
- link knee_ankle_left_link: geometry collision mesh filename=package://ros2_pkg/urdf/meshes/knee_ankle_left_link.STL; visual mesh filename=package://ros2_pkg/urdf/meshes/knee_ankle_left_link.STL
- link knee_ankle_right_link: geometry collision mesh filename=package://ros2_pkg/urdf/meshes/knee_ankle_right_link.STL; visual mesh filename=package://ros2_pkg/urdf/meshes/knee_ankle_right_link.STL
- link shoulder_elbow_left_link: geometry collision mesh filename=package://ros2_pkg/urdf/meshes/shoulder_elbow_left_link.STL; visual mesh filename=package://ros2_pkg/urdf/meshes/shoulder_elbow_left_link.STL
- link shoulder_elbow_right_link: geometry collision mesh filename=package://ros2_pkg/urdf/meshes/shoulder_elbow_right_link.STL; visual mesh filename=package://ros2_pkg/urdf/meshes/shoulder_elbow_right_link.STL
- link shoulder_shoulder_left_link: geometry collision mesh filename=package://ros2_pkg/urdf/meshes/shoulder_shoulder_left_link.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; visual mesh filename=package://ros2_pkg/urdf/meshes/shoulder_shoulder_left_link.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
- link shoulder_shoulder_right_link: geometry collision mesh filename=package://ros2_pkg/urdf/meshes/shoulder_shoulder_right_link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; visual mesh filename=package://ros2_pkg/urdf/meshes/shoulder_shoulder_right_link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

Commit message: fix urdf

File: Software/Ros2_WS/src/ros2_pkg/urdf/urdf/Robot.urdf (robot description, URDF)
Before this commit: robot Robot, 19 links, 18 joints
Links:
- link ankle_ankle_right_link: mass 0.0859210745449871 -> 0.085921074544987
- link hip_hip_right_link: mass 0.0244428963393534 -> 0.0244428963393535
- link knee_ankle_right_link: mass 0.0298519989099933 -> 0.0298519989099934
Joints:
- joint ankle_ankle_left_joint: origin xyz=0.0215 -0.0570000000000001 -0.0180000000000003 rpy=0 1.5707963267949 0 -> xyz=0.0215 -0.057 -0.018 rpy=0 1.5708 0
- joint ankle_ankle_right_joint: origin xyz=0.0214999999999963 -0.0569999999999992 -0.0215000000000082 rpy=0 1.5707963267949 0 -> xyz=0.0215 -0.057 -0.0215 rpy=0 1.5708 0
- joint base_hip_right_joint: origin xyz=0.035 -0.0205 -0.027 rpy=1.5708 0 0 -> xyz=0.0350000000000045 -0.0204999999999993 -0.027 rpy=1.5707963267949 0 0
- joint hip_knee_left_joint: origin xyz=0 -0.06 0 rpy=0 0 0 -> xyz=0 -0.0599999999999997 0 rpy=0 0 0
