Commit message: fix reward ppo

File: Software/MuJoCo_Training/assets/Robot.urdf (robot description, URDF)
Before this commit: robot Robot, 19 links, 18 joints
Links:
- link ankle_ankle_left_link: geometry collision mesh filename=/home/nckh/Desktop/NCKH_2026/Software/MuJoCo_Training/asset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; visual mesh filename=/home/nckh/Desktop/NCKH_2026/Software/MuJoCo_Training/asset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
- link ankle_ankle_right_link: geometry collision mesh filename=/home/nckh/Desktop/NCKH_2026/Software/MuJoCo_Training/asset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; visual mesh filename=/home/nckh/Desktop/NCKH_2026/Software/MuJoCo_Training/asset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
- link base_hip_left_link: geometry collision mesh filename=/home/nckh/Desktop/NCKH_2026/Software/MuJoCo_Training/asset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; visual mesh filename=/home/nckh/Desktop/NCKH_2026/Software/MuJoCo_Training/asset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
- link base_hip_middle_link: geometry collision mesh filename=/home/nckh/Desktop/NCKH_2026/Software/MuJoCo_Training/asset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; visual mesh filename=/home/nckh/Desktop/NCKH_2026/Software/MuJoCo_Training/asset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
- link base_hip_right_link: geometry collision mesh filename=/home/nckh/Desktop/NCKH_2026/Software/MuJoCo_Training/asset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; visual mesh filename=/home/nckh/Desktop/NCKH_2026/Software/MuJoCo_Training/asset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
- link base_link: geometry collision mesh filename=/home/nckh/Desktop/NCKH_2026/Software/MuJoCo_Training/asset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; visual mesh filename=/home/nckh/Desktop/NCKH_2026/Software/MuJoCo_Training/asset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
- link hip_head_link: geometry collision mesh filename=/home/nckh/Desktop/NCKH_2026/Software/MuJoCo_Training/asset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; visual mesh filename=/home/nckh/Desktop/NCKH_2026/Software/MuJoCo_Training/asset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
- link hip_hip_left_link: geometry collision mesh filename=/home/nckh/Desktop/NCKH_2026/Software/MuJoCo_Training/asset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; visual mesh filename=/home/nckh/Desktop/NCKH_2026/Software/MuJoCo_Training/asset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
- link hip_hip_right_link: geometry collision mesh filename=/home/nckh/Desktop/NCKH_2026/Software/MuJoCo_Training/asset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; visual mesh filename=/home/nckh/Desktop/NCKH_2026/Software/MuJoCo_Training/asset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
- link hip_knee_left_link: geometry collision mesh filename=/home/nckh/Desktop/NCKH_2026/Software/MuJoCo_Training/asset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; visual mesh filename=/home/nckh/Desktop/NCKH_2026/Software/MuJoCo_Training/asset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
- link hip_knee_right_link: geometry collision mesh filename=/home/nckh/Desktop/NCKH_2026/Software/MuJoCo_Training/asset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; visual mesh filename=/home/nckh/Desktop/NCKH_2026/Software/MuJoCo_Training/asset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
- link hip_shoulder_left_link: geometry collision mesh filename=/home/nckh/Desktop/NCKH_2026/Software/MuJoCo_Training/asset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; visual mesh filename=/home/nckh/Desktop/NCKH_2026/Software/MuJoCo_Training/asset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
- link hip_shoulder_right_link: geometry collision mesh filename=/home/nckh/Desktop/NCKH_2026/Software/MuJoCo_Training/asset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; visual mesh filename=/home/nckh/Desktop/NCKH_2026/Software/MuJoCo_Training/asset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
- link knee_ankle_left_link: geometry collision mesh filename=/home/nckh/Desktop/NCKH_2026/Software/MuJoCo_Training/asset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; visual mesh filename=/home/nckh/Desktop/NCKH_2026/Software/MuJoCo_Training/asset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
- link knee_ankle_right_link: geometry collision mesh filename=/home/nckh/Desktop/NCKH_2026/Software/MuJoCo_Training/asset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; visual mesh filename=/home/nckh/Desktop/NCKH_2026/Software/MuJoCo_Training/asset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
- link shoulder_elbow_left_link: geometry collision mesh filename=/home/nckh/Desktop/NCKH_2026/Software/MuJoCo_Training/asset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; visual mesh filename=/home/nckh/Desktop/NCKH_2026/Software/MuJoCo_Training/asset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
- link shoulder_elbow_right_link: geometry collision mesh filename=/home/nckh/Desktop/NCKH_2026/Software/MuJoCo_Training/asset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; visual mesh filename=/home/nckh/Desktop/NCKH_2026/Software/MuJoCo_Training/asset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
- link shoulder_shoulder_left_link: geometry collision mesh filename=/home/nckh/Desktop/NCKH_2026/Software/MuJoCo_Training/asset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; visual mesh filename=/home/nckh/Desktop/NCKH_2026/Software/MuJoCo_Training/asset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
- link shoulder_shoulder_right_link: geometry collision mesh filename=/home/nckh/Desktop/NCKH_2026/Software/MuJoCo_Training/asset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; visual mesh filename=/home/nckh/Desktop/NCKH_2026/Software/MuJoCo_Training/asset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

File: Software/Ros2_WS/install/ros2_pkg/share/ros2_pkg/urdf/humanoid_physics.xacro (robot description, xacro)
@@ -1 +1 @@
-/home/du/Desktop/NCKH_2026/Software/Ros2_WS/src/ros2_pkg/urdf/humanoid_physics.xacro
+/home/nckh/Desktop/NCKH_2026/Software/Ros2_WS/src/ros2_pkg/urdf/humanoid_physics.xacro

File: Software/Ros2_WS/install/ros2_pkg/share/ros2_pkg/urdf/main.xacro (robot description, xacro)
@@ -1 +1 @@
-/home/du/Desktop/NCKH_2026/Software/Ros2_WS/src/ros2_pkg/urdf/main.xacro
+/home/nckh/Desktop/NCKH_2026/Software/Ros2_WS/src/ros2_pkg/urdf/main.xacro

File: Software/Ros2_WS/install/ros2_pkg/share/ros2_pkg/urdf/main_turbo.xacro (robot description, xacro)
@@ -1 +1 @@
-/home/du/Desktop/NCKH_2026/Software/Ros2_WS/src/ros2_pkg/urdf/main_turbo.xacro
+/home/nckh/Desktop/NCKH_2026/Software/Ros2_WS/src/ros2_pkg/urdf/main_turbo.xacro

File: Software/Ros2_WS/src/ros2_pkg/urdf/humanoid_physics.xacro (robot description, xacro)
@@ -1,10 +1,10 @@
 <?xml version="1.0"?>
 <robot xmlns:xacro="http://www.ros.org/wiki/xacro">
-  <xacro:property name="petg_mu" value="0.8" />
+  <xacro:property name="petg_mu" value="0.6" />
   <xacro:property name="petg_kp" value="100000.0" />
   <xacro:property name="petg_kd" value="10.0" />
-  <xacro:property name="silicone_mu" value="0.99" />
+  <xacro:property name="silicone_mu" value="0.8" />
   <xacro:property name="silicone_kp" value="40000.0" />
-  <xacro:property name="silicone_kd" value="1200.0" />
+  <xacro:property name="silicone_kd" value="12.0" />
   <xacro:property name="silicone_thickness" value="0.002" />
   <xacro:macro name="setup_joint" params="joint_name">
@@ -47,13 +47,13 @@
     </gazebo>
     <xacro:setup_joint joint_name="base_hip_left_joint"/>
-    <xacro:make_controller joint_name="base_hip_left_joint"    p="1000" d="20"/>
+    <xacro:make_controller joint_name="base_hip_left_joint"    p="2000" d="20"/>
     <xacro:setup_joint joint_name="hip_hip_left_joint"/>
-    <xacro:make_controller joint_name="hip_hip_left_joint"     p="2000" d="30"/>
+    <xacro:make_controller joint_name="hip_hip_left_joint"     p="2000" d="20"/>
     <xacro:setup_joint joint_name="hip_knee_left_joint"/>
-    <xacro:make_controller joint_name="hip_knee_left_joint"    p="1000" d="20"/>
+    <xacro:make_controller joint_name="hip_knee_left_joint"    p="2000" d="20"/>
     <xacro:setup_joint joint_name="knee_ankle_left_joint"/>
-    <xacro:make_controller joint_name="knee_ankle_left_joint"  p="1000" d="20"/>
+    <xacro:make_controller joint_name="knee_ankle_left_joint"  p="2000" d="20"/>
     <xacro:setup_joint joint_name="ankle_ankle_left_joint"/>
-    <xacro:make_controller joint_name="ankle_ankle_left_joint" p="1000" d="20"/>
+    <xacro:make_controller joint_name="ankle_ankle_left_joint" p="2000" d="20"/>
     <gazebo reference="ankle_ankle_left_link">
       <mu1>${silicone_mu}</mu1>
@@ -63,13 +63,13 @@
     </gazebo>
     <xacro:setup_joint joint_name="base_hip_right_joint"/>
-    <xacro:make_controller joint_name="base_hip_right_joint"    p="1000" d="20"/>
+    <xacro:make_controller joint_name="base_hip_right_joint"    p="2000" d="20"/>
     <xacro:setup_joint joint_name="hip_hip_right_joint"/>
-    <xacro:make_controller joint_name="hip_hip_right_joint"     p="2000" d="30"/>
+    <xacro:make_controller joint_name="hip_hip_right_joint"     p="2000" d="20"/>
     <xacro:setup_joint joint_name="hip_knee_right_joint"/>
-    <xacro:make_controller joint_name="hip_knee_right_joint"    p="1000" d="20"/>
+    <xacro:make_controller joint_name="hip_knee_right_joint"    p="2000" d="20"/>
     <xacro:setup_joint joint_name="knee_ankle_right_joint"/>
-    <xacro:make_controller joint_name="knee_ankle_right_joint"  p="1000" d="20"/>
+    <xacro:make_controller joint_name="knee_ankle_right_joint"  p="2000" d="20"/>
     <xacro:setup_joint joint_name="ankle_ankle_right_joint"/>
-    <xacro:make_controller joint_name="ankle_ankle_right_joint" p="1000" d="20"/>
+    <xacro:make_controller joint_name="ankle_ankle_right_joint" p="2000" d="20"/>
     <gazebo reference="ankle_ankle_right_link">
       <mu1>${silicone_mu}</mu1>
