Commit message: fix uvc

File: Software/Ros2_WS/src/ros2_pkg/urdf/humanoid_physics.xacro (robot description, xacro)
@@ -1,34 +1,35 @@
 <?xml version="1.0"?>
 <robot xmlns:xacro="http://www.ros.org/wiki/xacro">
-  <xacro:property name="petg_mu1" value="1.5" />
-  <xacro:property name="petg_mu2" value="1.0" />
-  <xacro:property name="petg_kp" value="1000000.0" />
-  <xacro:property name="petg_kd" value="100.0" />
-  <!-- gan ma sat-->
+  <xacro:property name="petg_mu" value="0.7" />
+  <xacro:property name="petg_kp" value="100000.0" /> <xacro:property name="petg_kd" value="1.0" />
   <xacro:macro name="setup_link" params="link_name">
     <gazebo reference="${link_name}">
-      <mu1>${petg_mu1}</mu1>
-      <mu2>${petg_mu2}</mu2>
+      <mu1>${petg_mu}</mu1>
+      <mu2>${petg_mu}</mu2>
       <kp>${petg_kp}</kp>
       <kd>${petg_kd}</kd>
+      <auto_inertia_params><mass>0.15</mass></auto_inertia_params>
     </gazebo>
   </xacro:macro>
-  <!--them plugin-->
   <xacro:macro name="robot_brain">
     <gazebo>
-      <plugin
-        filename="gz-sim-joint-state-publisher-system"
-        name="gz::sim::systems::JointStatePublisher">
-        <update_rate>50</update_rate>
+      <plugin filename="gz-sim-joint-state-publisher-system" name="gz::sim::systems::JointStatePublisher">
+        <update_rate>100</update_rate>
       </plugin>
-      <plugin
-        filename="gz-sim-joint-trajectory-controller-system"
-        name="gz::sim::systems::JointTrajectoryController">
+      <plugin filename="gz-sim-joint-trajectory-controller-system" name="gz::sim::systems::JointTrajectoryController">
         <topic>/model/humanoid_robot/joint_trajectory</topic>
-      </plugin>
-      <plugin filename="gz-sim-imu-system" name="gz::sim::systems::Imu">
-      </plugin>
-      <plugin filename="gz-sim-scene-broadcaster-system" name="gz::sim::systems::SceneBroadcaster">
-      </plugin>
+        <gains joint_name="hip_knee_left_joint">    <p>5000</p> <d>50</d> <i_clamp>0</i_clamp> <max_force>6.0</max_force> </gains>
+        <gains joint_name="hip_knee_right_joint">   <p>5000</p> <d>50</d> <i_clamp>0</i_clamp> <max_force>6.0</max_force> </gains>
+        <gains joint_name="knee_ankle_left_joint">  <p>5000</p> <d>50</d> <i_clamp>0</i_clamp> <max_force>6.0</max_force> </gains>
+        <gains joint_name="knee_ankle_right_joint"> <p>5000</p> <d>50</d> <i_clamp>0</i_clamp> <max_force>6.0</max_force> </gains>
+        <gains joint_name="hip_hip_left_joint">     <p>5000</p> <d>50</d> <i_clamp>0</i_clamp> <max_force>6.0</max_force> </gains>
+        <gains joint_name="hip_hip_right_joint">    <p>5000</p> <d>50</d> <i_clamp>0</i_clamp> <max_force>6.0</max_force> </gains>
+        <gains joint_name="base_hip_left_joint">    <p>5000</p> <d>50</d> </gains>
+        <gains joint_name="base_hip_right_joint">   <p>5000</p> <d>50</d> </gains>
+        <gains joint_name="base_hip_middle_joint">  <p>5000</p> <d>50</d> </gains>
+        <gains joint_name="knee_knee_left_joint">   <p>5000</p> <d>50</d> </gains>
+        <gains joint_name="ankle_ankle_right_joint"><p>5000</p> <d>50</d> </gains>
+        </plugin>
+      <plugin filename="gz-sim-imu-system" name="gz::sim::systems::Imu"></plugin>
     </gazebo>
   </xacro:macro>
@@ -36,4 +37,6 @@
     <gazebo reference="${joint_name}">
       <implicitSpringDamper>true</implicitSpringDamper>
+      <friction>0.1</friction>
+      <damping>0.1</damping>
     </gazebo>
   </xacro:macro>

File: Software/Ros2_WS/src/ros2_pkg/urdf/main.xacro (robot description, xacro)
@@ -22,5 +22,11 @@
   <xacro:setup_link link_name="knee_ankle_right_link" />
   <xacro:setup_link link_name="ankle_ankle_right_link" />
-  <gazebo reference="base_link">
+  <xacro:setup_link link_name="hip_shoulder_left_link" />
+  <xacro:setup_link link_name="shoulder_shoulder_left_link" />
+  <xacro:setup_link link_name="shoulder_elbow_left_link" />
+  <xacro:setup_link link_name="hip_shoulder_right_link" />
+  <xacro:setup_link link_name="shoulder_shoulder_right_link" />
+  <xacro:setup_link link_name="shoulder_elbow_right_link" />
+  <gazebo reference="hip_head_link">
     <sensor name="imu_sensor" type="imu">
       <always_on>1</always_on>
@@ -31,9 +37,18 @@
   </gazebo>
   <xacro:robot_brain />
+  <xacro:setup_joint joint_name="base_hip_middle_joint" />
+  <xacro:setup_joint joint_name="base_hip_left_joint" />
+  <xacro:setup_joint joint_name="base_hip_right_joint" />
   <xacro:setup_joint joint_name="hip_hip_left_joint" />
   <xacro:setup_joint joint_name="hip_knee_left_joint" />
   <xacro:setup_joint joint_name="knee_ankle_left_joint" />
-  <xacro:setup_joint joint_name="hip_hip_right_joint" />
+  <xacro:setup_joint joint_name="knee_knee_left_joint" /> <xacro:setup_joint joint_name="hip_hip_right_joint" />
   <xacro:setup_joint joint_name="hip_knee_right_joint" />
   <xacro:setup_joint joint_name="knee_ankle_right_joint" />
+  <xacro:setup_joint joint_name="ankle_ankle_right_joint" /> <xacro:setup_joint joint_name="hip_shoulder_left_joint" />
+  <xacro:setup_joint joint_name="shoulder_shoulder_left_joint" />
+  <xacro:setup_joint joint_name="shoulder_elbow_left_joint" />
+  <xacro:setup_joint joint_name="hip_shoulder_right_joint" />
+  <xacro:setup_joint joint_name="shoulder_shoulder_right_joint" />
+  <xacro:setup_joint joint_name="shoulder_elbow_right_joint" />
 </robot>

File: Software/Ros2_WS/src/ros2_pkg/urdf/urdf/Robot.urdf (robot description, URDF)
Before this commit: robot Robot, 19 links, 18 joints
Joints:
- joint ankle_ankle_right_joint: limit lower=-1.2217 upper=1.2217 effort=1.08 velocity=6.16 -> lower=-1.2217 upper=1.2217 effort=2.5 velocity=6.16
- joint base_hip_left_joint: limit lower=-0.17453 upper=0.69813 effort=1.08 velocity=6.16 -> lower=-0.17453 upper=0.69813 effort=2.5 velocity=6.16
- joint base_hip_middle_joint: limit lower=-0.5236 upper=0.5236 effort=1.08 velocity=6.16 -> lower=-0.5236 upper=0.5236 effort=2.5 velocity=6.16
- joint base_hip_right_joint: limit lower=-0.69813 upper=0.17453 effort=1.08 velocity=6.16 -> lower=-0.69813 upper=0.17453 effort=2.5 velocity=6.16
- joint hip_hip_left_joint: limit lower=-0.5236 upper=0.69813 effort=1.08 velocity=6.16 -> lower=-0.5236 upper=0.69813 effort=2.5 velocity=6.16
- joint hip_hip_right_joint: limit lower=-0.69813 upper=0.5236 effort=1.08 velocity=6.16 -> lower=-0.69813 upper=0.5236 effort=2.5 velocity=6.16
- joint hip_knee_left_joint: limit lower=-1.3963 upper=1.3963 effort=1.08 velocity=6.16 -> lower=-1.3963 upper=1.3963 effort=2.5 velocity=6.16
- joint hip_knee_right_joint: limit lower=-1.3963 upper=1.3963 effort=1.08 velocity=6.16 -> lower=-1.3963 upper=1.3963 effort=2.5 velocity=6.16
- joint hip_shoulder_left_joint: limit lower=-1.2217 upper=0.17453 effort=1.08 velocity=6.16 -> lower=-1.2217 upper=0.17453 effort=2.5 velocity=6.16
- joint hip_shoulder_right_joint: limit lower=-0.17453 upper=1.2217 effort=1.08 velocity=6.16 -> lower=-0.17453 upper=1.2217 effort=2.5 velocity=6.16
- joint knee_ankle_left_joint: limit lower=-0.34907 upper=0.69813 effort=1.08 velocity=6.16 -> lower=-0.34907 upper=0.69813 effort=2.5 velocity=6.16
- joint knee_ankle_right_joint: limit lower=-0.69813 upper=0.34907 effort=1.08 velocity=6.16 -> lower=-0.69813 upper=0.34907 effort=2.5 velocity=6.16
- joint knee_knee_left_joint: limit lower=-1.2217 upper=1.2217 effort=1.08 velocity=6.16 -> lower=-1.2217 upper=1.2217 effort=2.5 velocity=6.16
- joint shoulder_elbow_left_joint: limit lower=-1.3963 upper=1.3963 effort=1.08 velocity=6.16 -> lower=-1.3963 upper=1.3963 effort=2.5 velocity=6.16
- joint shoulder_elbow_right_joint: limit lower=-1.3963 upper=1.3963 effort=1.08 velocity=6.16 -> lower=-1.3963 upper=1.3963 effort=2.5 velocity=6.16
- joint shoulder_shoulder_left_joint: limit lower=-1.0472 upper=1.0472 effort=1.08 velocity=6.16 -> lower=-1.0472 upper=1.0472 effort=2.5 velocity=6.16
- joint shoulder_shoulder_right_joint: limit lower=-1.0472 upper=1.0472 effort=1.08 velocity=6.16 -> lower=-1.0472 upper=1.0472 effort=2.5 velocity=6.16

Commit message: fix rl

File: Software/Ros2_WS/src/ros2_pkg/urdf/humanoid_physics.xacro (robot description, xacro)
@@ -4,4 +4,10 @@
   <xacro:property name="petg_kp" value="1000000.0" />
   <xacro:property name="petg_kd" value="100.0" />
+  <!-- Silicone pad properties (for ankle soles) -->
+  <!-- Increased defaults to reduce slipping; tune if needed -->
+  <xacro:property name="silicone_mu" value="6.0" />
+  <xacro:property name="silicone_kp" value="5000000.0" />
+  <xacro:property name="silicone_kd" value="500.0" />
+  <xacro:property name="silicone_thickness" value="0.002" /> <!-- meters (2 mm) -->
   <xacro:macro name="setup_link" params="link_name">
     <gazebo reference="${link_name}">
@@ -54,4 +60,15 @@
     <xacro:make_controller joint_name="knee_ankle_left_joint"  p="8000" d="100"/>
     <xacro:make_controller joint_name="ankle_ankle_left_joint" p="8000" d="100"/>
+    <!-- Add silicone high-friction pad to left ankle link (simulated via higher mu/kp/kd) -->
+    <gazebo reference="ankle_ankle_left_link">
+      <!-- friction coefficients (mu1, mu2) increased to simulate sticky silicone -->
+      <mu1>${silicone_mu}</mu1>
+      <mu2>${silicone_mu}</mu2>
+      <!-- contact stiffness/damping tuned for soft pad -->
+      <kp>${silicone_kp}</kp>
+      <kd>${silicone_kd}</kd>
+      <!-- note: thickness is for documentation; to add geometry, modify URDF collision separately -->
+      <silicone_thickness>${silicone_thickness}</silicone_thickness>
+    </gazebo>
     <xacro:setup_joint joint_name="base_hip_right_joint"/>
     <xacro:setup_joint joint_name="hip_hip_right_joint"/>
@@ -64,4 +81,12 @@
     <xacro:make_controller joint_name="knee_ankle_right_joint"  p="8000" d="100"/>
     <xacro:make_controller joint_name="ankle_ankle_right_joint" p="8000" d="100"/>
+    <!-- Add silicone high-friction pad to right ankle link -->
+    <gazebo reference="ankle_ankle_right_link">
+      <mu1>${silicone_mu}</mu1>
+      <mu2>${silicone_mu}</mu2>
+      <kp>${silicone_kp}</kp>
+      <kd>${silicone_kd}</kd>
+      <silicone_thickness>${silicone_thickness}</silicone_thickness>
+    </gazebo>
     <xacro:setup_joint joint_name="base_hip_middle_joint"/>
     <xacro:make_controller joint_name="base_hip_middle_joint"   p="8000" d="100"/>

Commit message: fix rl

File: Software/Ros2_WS/src/ros2_pkg/urdf/humanoid_physics.xacro (robot description, xacro)
@@ -1,13 +1,18 @@
 <?xml version="1.0"?>
 <robot xmlns:xacro="http://www.ros.org/wiki/xacro">
-  <xacro:property name="petg_mu" value="1.0" />
-  <xacro:property name="petg_kp" value="1000000.0" />
-  <xacro:property name="petg_kd" value="100.0" />
-  <!-- Silicone pad properties (for ankle soles) -->
-  <!-- Increased defaults to reduce slipping; tune if needed -->
-  <xacro:property name="silicone_mu" value="6.0" />
-  <xacro:property name="silicone_kp" value="5000000.0" />
-  <xacro:property name="silicone_kd" value="500.0" />
-  <xacro:property name="silicone_thickness" value="0.002" /> <!-- meters (2 mm) -->
+  <xacro:property name="petg_mu" value="0.8" />
+  <xacro:property name="petg_kp" value="100000.0" />
+  <xacro:property name="petg_kd" value="10.0" />
+  <xacro:property name="silicone_mu" value="0.99" />
+  <xacro:property name="silicone_kp" value="40000.0" />
+  <xacro:property name="silicone_kd" value="1200.0" />
+  <xacro:property name="silicone_thickness" value="0.002" />
+  <xacro:macro name="setup_joint" params="joint_name">
+    <gazebo reference="${joint_name}">
+      <implicitSpringDamper>true</implicitSpringDamper>
+      <friction>0.2</friction>
+      <damping>0.1</damping>
+    </gazebo>
+  </xacro:macro>
   <xacro:macro name="setup_link" params="link_name">
     <gazebo reference="${link_name}">
@@ -16,13 +21,4 @@
       <kp>${petg_kp}</kp>
       <kd>${petg_kd}</kd>
-    </gazebo>
-  </xacro:macro>
-  <xacro:macro name="setup_joint" params="joint_name">
-    <gazebo reference="${joint_name}">
-      <implicitSpringDamper>true</implicitSpringDamper>
-      <springStiffness>0.0</springStiffness>
-      <springReference>0.0</springReference>
-      <friction>1.5</friction>
-      <damping>1.0</damping>
     </gazebo>
   </xacro:macro>
@@ -34,10 +30,10 @@
         <topic>/model/humanoid_robot/joint/${joint_name}/cmd_pos</topic>
         <p_gain>${p}</p_gain>
-        <i_gain>0.5</i_gain>
+        <i_gain>0.01</i_gain>
         <d_gain>${d}</d_gain>
-        <i_max>10</i_max>
-        <i_min>-10</i_min>
-        <cmd_max>200.0</cmd_max>
-        <cmd_min>-200.0</cmd_min>
+        <i_max>1</i_max>
+        <i_min>-1</i_min>
+        <cmd_max>2.5</cmd_max>
+        <cmd_min>-2.5</cmd_min>
       </plugin>
     </gazebo>
@@ -51,35 +47,29 @@
     </gazebo>
     <xacro:setup_joint joint_name="base_hip_left_joint"/>
+    <xacro:make_controller joint_name="base_hip_left_joint"    p="1000" d="20"/>
     <xacro:setup_joint joint_name="hip_hip_left_joint"/>
+    <xacro:make_controller joint_name="hip_hip_left_joint"     p="2000" d="30"/>
     <xacro:setup_joint joint_name="hip_knee_left_joint"/>
+    <xacro:make_controller joint_name="hip_knee_left_joint"    p="1000" d="20"/>
     <xacro:setup_joint joint_name="knee_ankle_left_joint"/>
+    <xacro:make_controller joint_name="knee_ankle_left_joint"  p="1000" d="20"/>
     <xacro:setup_joint joint_name="ankle_ankle_left_joint"/>
-    <xacro:make_controller joint_name="base_hip_left_joint"    p="8000" d="100"/>
-    <xacro:make_controller joint_name="hip_hip_left_joint"     p="8000" d="100"/>
-    <xacro:make_controller joint_name="hip_knee_left_joint"    p="8000" d="100"/>
-    <xacro:make_controller joint_name="knee_ankle_left_joint"  p="8000" d="100"/>
-    <xacro:make_controller joint_name="ankle_ankle_left_joint" p="8000" d="100"/>
-    <!-- Add silicone high-friction pad to left ankle link (simulated via higher mu/kp/kd) -->
+    <xacro:make_controller joint_name="ankle_ankle_left_joint" p="1000" d="20"/>
     <gazebo reference="ankle_ankle_left_link">
-      <!-- friction coefficients (mu1, mu2) increased to simulate sticky silicone -->
       <mu1>${silicone_mu}</mu1>
       <mu2>${silicone_mu}</mu2>
-      <!-- contact stiffness/damping tuned for soft pad -->
       <kp>${silicone_kp}</kp>
       <kd>${silicone_kd}</kd>
-      <!-- note: thickness is for documentation; to add geometry, modify URDF collision separately -->
-      <silicone_thickness>${silicone_thickness}</silicone_thickness>
     </gazebo>
     <xacro:setup_joint joint_name="base_hip_right_joint"/>
+    <xacro:make_controller joint_name="base_hip_right_joint"    p="1000" d="20"/>
     <xacro:setup_joint joint_name="hip_hip_right_joint"/>
+    <xacro:make_controller joint_name="hip_hip_right_joint"     p="2000" d="30"/>
     <xacro:setup_joint joint_name="hip_knee_right_joint"/>
+    <xacro:make_controller joint_name="hip_knee_right_joint"    p="1000" d="20"/>
     <xacro:setup_joint joint_name="knee_ankle_right_joint"/>
+    <xacro:make_controller joint_name="knee_ankle_right_joint"  p="1000" d="20"/>
     <xacro:setup_joint joint_name="ankle_ankle_right_joint"/>
-    <xacro:make_controller joint_name="base_hip_right_joint"    p="8000" d="100"/>
-    <xacro:make_controller joint_name="hip_hip_right_joint"     p="8000" d="100"/>
-    <xacro:make_controller joint_name="hip_knee_right_joint"    p="8000" d="100"/>
-    <xacro:make_controller joint_name="knee_ankle_right_joint"  p="8000" d="100"/>
-    <xacro:make_controller joint_name="ankle_ankle_right_joint" p="8000" d="100"/>
-    <!-- Add silicone high-friction pad to right ankle link -->
+    <xacro:make_controller joint_name="ankle_ankle_right_joint" p="1000" d="20"/>
     <gazebo reference="ankle_ankle_right_link">
       <mu1>${silicone_mu}</mu1>
@@ -87,20 +77,19 @@
       <kp>${silicone_kp}</kp>
       <kd>${silicone_kd}</kd>
-      <silicone_thickness>${silicone_thickness}</silicone_thickness>
     </gazebo>
     <xacro:setup_joint joint_name="base_hip_middle_joint"/>
-    <xacro:make_controller joint_name="base_hip_middle_joint"   p="8000" d="100"/>
+    <xacro:make_controller joint_name="base_hip_middle_joint"   p="300" d="5"/>
     <xacro:setup_joint joint_name="hip_shoulder_left_joint"/>
+    <xacro:make_controller joint_name="hip_shoulder_left_joint"      p="200" d="5"/>
     <xacro:setup_joint joint_name="shoulder_shoulder_left_joint"/>
+    <xacro:make_controller joint_name="shoulder_shoulder_left_joint" p="200" d="5"/>
     <xacro:setup_joint joint_name="shoulder_elbow_left_joint"/>
-    <xacro:make_controller joint_name="hip_shoulder_left_joint"      p="8000" d="100"/>
-    <xacro:make_controller joint_name="shoulder_shoulder_left_joint" p="8000" d="100"/>
-    <xacro:make_controller joint_name="shoulder_elbow_left_joint"    p="8000" d="100"/>
+    <xacro:make_controller joint_name="shoulder_elbow_left_joint"    p="200" d="5"/>
     <xacro:setup_joint joint_name="hip_shoulder_right_joint"/>
+    <xacro:make_controller joint_name="hip_shoulder_right_joint"      p="200" d="5"/>
     <xacro:setup_joint joint_name="shoulder_shoulder_right_joint"/>
+    <xacro:make_controller joint_name="shoulder_shoulder_right_joint" p="200" d="5"/>
     <xacro:setup_joint joint_name="shoulder_elbow_right_joint"/>
-    <xacro:make_controller joint_name="hip_shoulder_right_joint"      p="8000" d="100"/>
-    <xacro:make_controller joint_name="shoulder_shoulder_right_joint" p="8000" d="100"/>
-    <xacro:make_controller joint_name="shoulder_elbow_right_joint"    p="8000" d="100"/>
+    <xacro:make_controller joint_name="shoulder_elbow_right_joint"    p="200" d="5"/>
   </xacro:macro>
 </robot>
