Commit message: fix phase 1 cpg

File: Software/Ros2_WS_v2/src/ros2_pkg_v2/urdf/humanoid_physics.xacro (robot description, xacro)
@@ -4,5 +4,5 @@
        VẬT LIỆU PETG: Dùng cho tất cả link NGOẠI TRỪ bàn chân
        ============================================================ -->
-  <xacro:property name="petg_mu" value="0.7" />
+  <xacro:property name="petg_mu" value="0.99" />
   <xacro:property name="petg_kp" value="100000.0" />
   <xacro:property name="petg_kd" value="10.0" />
